Commit message: updated README.md

File: avatar_gripper_description/urdf/avatar_gripper_3f.urdf (robot description, URDF)
Before this commit: robot avatar_gripper_3f_model, 13 links, 12 joints
Links:
- link right_gripper_base: geometry visual mesh filename=package://avatar_gripper_description/meshes/gripper_base.obj
- link right_index_base_connector: geometry visual mesh filename=package://avatar_gripper_description/meshes/index_base_conn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
- link right_index_fingertip: geometry collision mesh filename=package://avatar_gripper_description/meshes/index_fingertip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; visual mesh filename=package://avatar_gripper_description/meshes/index_fingertip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
- link right_index_knuckle: geometry collision mesh filename=package://avatar_gripper_description/meshes/index_knuckle.o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; visual mesh filename=package://avatar_gripper_description/meshes/index_knuckle.o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
- link right_middle_fingertip: geometry collision mesh filename=package://avatar_gripper_description/meshes/index_fingertip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; visual mesh filename=package://avatar_gripper_description/meshes/index_fingertip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
- link right_middle_knuckle: geometry collision mesh filename=package://avatar_gripper_description/meshes/index_knuckle.o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; visual mesh filename=package://avatar_gripper_description/meshes/index_knuckle.o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
- link right_thumb_base: geometry collision mesh filename=package://avatar_gripper_description/meshes/thumb_base_extr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; visual mesh filename=package://avatar_gripper_description/meshes/thumb_base_extr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
- link right_thumb_finger: geometry collision mesh filename=package://avatar_gripper_description/meshes/thumb_fingertip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; visual mesh filename=package://avatar_gripper_description/meshes/thumb_fingertip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
- link right_thumb_knuckle: geometry collision mesh filename=package://avatar_gripper_description/meshes/thumb_knuckle.o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; visual mesh filename=package://avatar_gripper_description/meshes/thumb_knuckle.o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
- link right_thumb_swivel_link: geometry visual mesh filename=package://avatar_gripper_description/meshes/thumb_swivel_li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
Joints:
- joint right_index_fingertip_joint: mimic joint=right_index_flex_motor_joint multiplier=-0.40 -> joint=right_index_flex_motor_joint multiplier=0.40
- joint right_index_flex_motor_joint: limit lower=0 upper=1.0 effort=1000 velocity=2.0 -> lower=-1.0 upper=0.0 effort=1000 velocity=2.0
- joint right_index_knuckle_joint: mimic joint=right_index_flex_motor_joint multiplier=-1 -> joint=right_index_flex_motor_joint multiplier=1
- joint right_thumb_finger_joint: mimic joint=right_thumb_flex_motor_joint multiplier=-0.6007 -> joint=right_thumb_flex_motor_joint multiplier=0.6007
- joint right_thumb_flex_motor_joint: limit lower=0 upper=1.0 effort=1000 velocity=2.0 -> lower=-1.0 upper=0.0 effort=1000 velocity=2.0
- joint right_thumb_knuckle_joint: mimic joint=right_thumb_flex_motor_joint multiplier=-0.5702 -> joint=right_thumb_flex_motor_joint multiplier=0.5702
- joint right_thumb_swivel_joint: mimic joint=right_thumb_swivel_motor_joint multiplier=0.6075 offset=0.43 -> joint=right_thumb_swivel_motor_joint multiplier=-0.6075 offset=0.43
- joint right_thumb_swivel_motor_joint: limit lower=0 upper=2.0 effort=1000 velocity=2.0 -> lower=-2.0 upper=0.0 effort=1000 velocity=2.0
