Commit message: minor bug fix

File: avatar_gripper_description/urdf/avatar_gripper_3f_macro_nomimic.xacro (robot description, xacro)
@@ -185,4 +185,7 @@
       </visual>
       <collision>
+        <geometry>
+          <mesh filename="package://avatar_gripper_description/meshes/${prefix}/index_fingertip.obj"/>
+        </geometry>
         <origin xyz="0 0 0" rpy="0 0 0"/>
       </collision>

File: avatar_robot_description/franka/common/base.xacro (robot description, xacro)
@@ -44,5 +44,5 @@
 			</geometry>
 			<material name="Mat Black 1">
-				<color rgba  <!-- <xacro:avatar_gripper_3f prefix="$(arg pref)"/>; -->="0.1 0.1 0.1 1.0"/>
+				<color rgba="0.1 0.1 0.1 1.0"/>
 			</material>
 		</visual>
