Commit message: renaming and minor tunings

File: avatar_gripper_description/urdf/avatar_gripper_3f.xacro (robot description, xacro)
@@ -1,5 +1,13 @@
 <?xml version="1.0"?>
 <robot name="avatar_gripper_3f_model" xmlns:xacro="http://ros.org/wiki/xacro">
-  <xacro:include filename="$(find avatar_description)/urdf/avatar_gripper_3f_macro.xacro" />
-  <xacro:avatar_gripper_3f prefix=""/>
+  <xacro:include filename="$(find avatar_gripper_description)/urdf/avatar_gripper_3f_macro.xacro" />
+  <xacro:avatar_gripper_3f prefix="right"/>
+  <!-- <xacro:macro name="attach_gripper" params="connected_to:='' arm_id:='panda' rpy:='0 0 0' xyz:='0 0 0'">
+    <xacro:unless value="${connected_to == ''}">
+      <joint name="${arm_id}_gripper_joint" type="fixed">
+        <parent link="${connected_to}" />
+        <child link="${arm_id}_hand" />
+        <origin xyz="${xyz}" rpy="${rpy}" />
+      </joint>
+    </xacro:unless>     -->
 </robot>

File: avatar_gripper_description/urdf/avatar_gripper_3f_macro.xacro (robot description, xacro)
@@ -10,5 +10,5 @@
         <origin xyz="0 0 0" rpy="0 0 0"/>
         <geometry>
-          <mesh filename="package://avatar_description/meshes/gripper_base.obj"/>
+          <mesh filename="package://avatar_gripper_description/meshes/gripper_base.obj"/>
         </geometry>
         <material name="">
@@ -27,14 +27,14 @@
         <origin xyz="0 0 0" rpy="0 0 0"/>
         <geometry>
-          <mesh filename="package://avatar_description/meshes/thumb_base_extra.obj"/>
-        </geometry>
-        <material name="">
-          <color rgba="0.9 0.9 0.9 1"/>
-        </material>
-      </visual>
-      <collision>
-        <origin xyz="0 0 0" rpy="0 0 0"/>
-        <geometry>
-          <mesh filename="package://avatar_description/meshes/thumb_base_extra.obj"/>
+          <mesh filename="package://avatar_gripper_description/meshes/thumb_base_extra.obj"/>
+        </geometry>
+        <material name="">
+          <color rgba="0.9 0.9 0.9 1"/>
+        </material>
+      </visual>
+      <collision>
+        <origin xyz="0 0 0" rpy="0 0 0"/>
+        <geometry>
+          <mesh filename="package://avatar_gripper_description/meshes/thumb_base_extra.obj"/>
         </geometry>
       </collision>
@@ -50,14 +50,14 @@
         <origin xyz="0 0 0" rpy="0 0 0"/>
         <geometry>
-          <mesh filename="package://avatar_description/meshes/thumb_knuckle.obj"/>
-        </geometry>
-        <material name="">
-          <color rgba="0.9 0.9 0.9 1"/>
-        </material>
-      </visual>
-      <collision>
-        <origin xyz="0 0 0" rpy="0 0 0"/>
-        <geometry>
-          <mesh filename="package://avatar_description/meshes/thumb_knuckle.obj"/>
+          <mesh filename="package://avatar_gripper_description/meshes/thumb_knuckle.obj"/>
+        </geometry>
+        <material name="">
+          <color rgba="0.9 0.9 0.9 1"/>
+        </material>
+      </visual>
+      <collision>
+        <origin xyz="0 0 0" rpy="0 0 0"/>
+        <geometry>
+          <mesh filename="package://avatar_gripper_description/meshes/thumb_knuckle.obj"/>
         </geometry>
       </collision>
@@ -73,14 +73,14 @@
         <origin xyz="0 0 0" rpy="0 0 0"/>
         <geometry>
-          <mesh filename="package://avatar_description/meshes/thumb_fingertip.obj"/>
-        </geometry>
-        <material name="">
-          <color rgba="0.9 0.9 0.9 1"/>
-        </material>
-      </visual>
-      <collision>
-        <origin xyz="0 0 0" rpy="0 0 0"/>
-        <geometry>
-          <mesh filename="package://avatar_description/meshes/thumb_fingertip.obj"/>
+          <mesh filename="package://avatar_gripper_description/meshes/thumb_fingertip.obj"/>
+        </geometry>
+        <material name="">
+          <color rgba="0.9 0.9 0.9 1"/>
+        </material>
+      </visual>
+      <collision>
+        <origin xyz="0 0 0" rpy="0 0 0"/>
+        <geometry>
+          <mesh filename="package://avatar_gripper_description/meshes/thumb_fingertip.obj"/>
         </geometry>
       </collision>
@@ -92,5 +92,5 @@
         <origin xyz="0 0 0" rpy="0 0 0"/>
         <geometry>
-          <mesh filename="package://avatar_description/meshes/index_base_connector.obj"/>
+          <mesh filename="package://avatar_gripper_description/meshes/index_base_connector.obj"/>
         </geometry>
         <material name="">
@@ -109,14 +109,14 @@
         <origin xyz="0 0 0" rpy="0 0 0"/>
         <geometry>
-          <mesh filename="package://avatar_description/meshes/index_knuckle.obj"/>
-        </geometry>
-        <material name="">
-          <color rgba="0.9 0.9 0.9 1"/>
-        </material>
-      </visual>
-      <collision>
-        <origin xyz="0 0 0" rpy="0 0 0"/>
-        <geometry>
-          <mesh filename="package://avatar_description/meshes/index_knuckle.obj"/>
+          <mesh filename="package://avatar_gripper_description/meshes/index_knuckle.obj"/>
+        </geometry>
+        <material name="">
+          <color rgba="0.9 0.9 0.9 1"/>
+        </material>
+      </visual>
+      <collision>
+        <origin xyz="0 0 0" rpy="0 0 0"/>
+        <geometry>
+          <mesh filename="package://avatar_gripper_description/meshes/index_knuckle.obj"/>
         </geometry>
       </collision>
@@ -132,14 +132,14 @@
         <origin xyz="0 0 0" rpy="0 0 0"/>
         <geometry>
-          <mesh filename="package://avatar_description/meshes/index_fingertip.obj"/>
-        </geometry>
-        <material name="">
-          <color rgba="0.9 0.9 0.9 1"/>
-        </material>
-      </visual>
-      <collision>
-        <origin xyz="0 0 0" rpy="0 0 0"/>
-        <geometry>
-          <mesh filename="package://avatar_description/meshes/index_fingertip.obj"/>
+          <mesh filename="package://avatar_gripper_description/meshes/index_fingertip.obj"/>
+        </geometry>
+        <material name="">
+          <color rgba="0.9 0.9 0.9 1"/>
+        </material>
+      </visual>
+      <collision>
+        <origin xyz="0 0 0" rpy="0 0 0"/>
+        <geometry>
+          <mesh filename="package://avatar_gripper_description/meshes/index_fingertip.obj"/>
         </geometry>
       </collision>
@@ -155,14 +155,14 @@
         <origin xyz="0 0 0" rpy="0 0 0"/>
         <geometry>
-          <mesh filename="package://avatar_description/meshes/index_knuckle.obj"/>
-        </geometry>
-        <material name="">
-          <color rgba="0.9 0.9 0.9 1"/>
-        </material>
-      </visual>
-      <collision>
-        <origin xyz="0 0 0" rpy="0 0 0"/>
-        <geometry>
-          <mesh filename="package://avatar_description/meshes/index_knuckle.obj"/>
+          <mesh filename="package://avatar_gripper_description/meshes/index_knuckle.obj"/>
+        </geometry>
+        <material name="">
+          <color rgba="0.9 0.9 0.9 1"/>
+        </material>
+      </visual>
+      <collision>
+        <origin xyz="0 0 0" rpy="0 0 0"/>
+        <geometry>
+          <mesh filename="package://avatar_gripper_description/meshes/index_knuckle.obj"/>
         </geometry>
       </collision>
@@ -178,14 +178,14 @@
         <origin xyz="0 0 0" rpy="0 0 0"/>
         <geometry>
-          <mesh filename="package://avatar_description/meshes/index_fingertip.obj"/>
-        </geometry>
-        <material name="">
-          <color rgba="0.9 0.9 0.9 1"/>
-        </material>
-      </visual>
-      <collision>
-        <origin xyz="0 0 0" rpy="0 0 0"/>
-        <geometry>
-          <mesh filename="package://avatar_description/meshes/index_fingertip.obj"/>
+          <mesh filename="package://avatar_gripper_description/meshes/index_fingertip.obj"/>
+        </geometry>
+        <material name="">
+          <color rgba="0.9 0.9 0.9 1"/>
+        </material>
+      </visual>
+      <collision>
+        <origin xyz="0 0 0" rpy="0 0 0"/>
+        <geometry>
+          <mesh filename="package://avatar_gripper_description/meshes/index_fingertip.obj"/>
         </geometry>
       </collision>
@@ -197,5 +197,5 @@
         <origin xyz="0 0 0" rpy="0 0 0"/>
         <geometry>
-          <mesh filename="package://avatar_description/meshes/thumb_swivel_link.obj"/>
+          <mesh filename="package://avatar_gripper_description/meshes/thumb_swivel_link.obj"/>
         </geometry>
         <material name="">
@@ -213,5 +213,5 @@
       <axis xyz="0 1 0"/>
       <limit lower="-1.0" upper="0.4" velocity="2.0" effort="1000" />
-      <mimic joint="${prefix}_thumb_flex_motor_joint" offsite="0" multiplier="-0.5702"/>
+      <mimic joint="${prefix}_thumb_flex_motor_joint" offsite="0" multiplier="0.5702"/>
     </joint>
   </xacro:macro>
@@ -223,5 +223,5 @@
       <axis xyz="0 1 0"/>
       <limit lower="-0.8" upper="0" velocity="2.0" effort="1000" />
-      <mimic joint="${prefix}_thumb_flex_motor_joint" offsite="0" multiplier="-0.6007"/>
+      <mimic joint="${prefix}_thumb_flex_motor_joint" offsite="0" multiplier="0.6007"/>
     </joint>
   </xacro:macro>
@@ -240,5 +240,5 @@
       <axis xyz="0 0 1"/>
       <limit lower="0" upper="1.7" velocity="2.0" effort="1000" />
-      <mimic joint="${prefix}_thumb_swivel_motor_joint" offset="0.43" multiplier="0.6075"/>
+      <mimic joint="${prefix}_thumb_swivel_motor_joint" offset="0.43" multiplier="-0.6075"/>
     </joint>
   </xacro:macro>
@@ -250,5 +250,5 @@
       <axis xyz="0 0 1"/>
       <limit lower="-0.8" upper="0" velocity="2.0" effort="1000" />
-      <mimic joint="${prefix}_index_flex_motor_joint" offsite="0" multiplier="-1"/>
+      <mimic joint="${prefix}_index_flex_motor_joint" offsite="0" multiplier="1"/>
     </joint>
   </xacro:macro>
@@ -260,5 +260,5 @@
       <axis xyz="0 0 1"/>
       <limit lower="-0.8" upper="0" velocity="2.0" effort="1000" />
-      <mimic joint="${prefix}_index_flex_motor_joint" offsite="0" multiplier="-0.40"/>
+      <mimic joint="${prefix}_index_flex_motor_joint" offsite="0" multiplier="0.40"/>
     </joint>
   </xacro:macro>
@@ -312,5 +312,5 @@
       <child link="${prefix}_index_flex_motor"/>
       <axis xyz="0 0 1"/>
-      <limit lower="0" upper="1.0" velocity="2.0" effort="1000" />
+      <limit lower="-1.0" upper="0.0" velocity="2.0" effort="1000" />
     </joint>
   </xacro:macro>
@@ -321,5 +321,5 @@
       <child link="${prefix}_thumb_flex_motor"/>
       <axis xyz="0 0 1"/>
-      <limit lower="0" upper="1.0" velocity="2.0" effort="1000" />
+      <limit lower="-1.0" upper="0.0" velocity="2.0" effort="1000" />
     </joint>
   </xacro:macro>
@@ -330,33 +330,33 @@
       <child link="${prefix}_thumb_swivel_motor"/>
       <axis xyz="0 0 1"/>
-      <limit lower="0" upper="2.0" velocity="2.0" effort="1000" />
+      <limit lower="-2.0" upper="0.0" velocity="2.0" effort="1000" />
     </joint>
   </xacro:macro>
   <xacro:macro name="avatar_gripper_3f" params="prefix">
-    <xacro:thumb_base_link prefix="right"/>
-    <xacro:thumb_knuckle_link prefix="right"/>
-    <xacro:thumb_knuckle_joint prefix="right"/>
-    <xacro:thumb_finger_link prefix="right"/>
-    <xacro:thumb_finger_joint prefix="right"/>
-    <xacro:thumb_swivel_link prefix="right"/>
-    <xacro:thumb_swivel_joint prefix="right"/>
-    <xacro:thumb_base_swivel_joint prefix="right"/>
-    <xacro:index_base_connector prefix="right"/>
-    <xacro:index_knuckle prefix="right"/>
-    <xacro:index_knuckle_joint prefix="right"/>
-    <xacro:index_fingertip prefix="right"/>
-    <xacro:index_fingertip_joint prefix="right"/>
-    <xacro:middle_knuckle prefix="right"/>
-    <xacro:middle_knuckle_joint prefix="right"/>
-    <xacro:middle_fingertip prefix="right"/>
-    <xacro:middle_fingertip_joint prefix="right"/>
-    <xacro:gripper_base_link prefix="right"/>
-    <xacro:gripper_base_joint prefix="right"/>
-    <xacro:motor_link prefix="right" actuation="thumb_flex"/>
-    <xacro:thumb_flex_motor_joint prefix="right"/>
-    <xacro:motor_link prefix="right" actuation="thumb_swivel"/>
-    <xacro:thumb_swivel_motor_joint prefix="right"/>
-    <xacro:motor_link prefix="right" actuation="index_flex"/>
-    <xacro:index_flex_motor_joint prefix="right"/>
+    <xacro:thumb_base_link prefix="${prefix}"/>
+    <xacro:thumb_knuckle_link prefix="${prefix}"/>
+    <xacro:thumb_knuckle_joint prefix="${prefix}"/>
+    <xacro:thumb_finger_link prefix="${prefix}"/>
+    <xacro:thumb_finger_joint prefix="${prefix}"/>
+    <xacro:thumb_swivel_link prefix="${prefix}"/>
+    <xacro:thumb_swivel_joint prefix="${prefix}"/>
+    <xacro:thumb_base_swivel_joint prefix="${prefix}"/>
+    <xacro:index_base_connector prefix="${prefix}"/>
+    <xacro:index_knuckle prefix="${prefix}"/>
+    <xacro:index_knuckle_joint prefix="${prefix}"/>
+    <xacro:index_fingertip prefix="${prefix}"/>
+    <xacro:index_fingertip_joint prefix="${prefix}"/>
+    <xacro:middle_knuckle prefix="${prefix}"/>
+    <xacro:middle_knuckle_joint prefix="${prefix}"/>
+    <xacro:middle_fingertip prefix="${prefix}"/>
+    <xacro:middle_fingertip_joint prefix="${prefix}"/>
+    <xacro:gripper_base_link prefix="${prefix}"/>
+    <xacro:gripper_base_joint prefix="${prefix}"/>
+    <xacro:motor_link prefix="${prefix}" actuation="thumb_flex"/>
+    <xacro:thumb_flex_motor_joint prefix="${prefix}"/>
+    <xacro:motor_link prefix="${prefix}" actuation="thumb_swivel"/>
+    <xacro:thumb_swivel_motor_joint prefix="${prefix}"/>
+    <xacro:motor_link prefix="${prefix}" actuation="index_flex"/>
+    <xacro:index_flex_motor_joint prefix="${prefix}"/>
   </xacro:macro>
 </robot>

Commit message: connected the gripper with the panda arm

File: avatar_gripper_description/urdf/avatar_gripper_3f.xacro (robot description, xacro)
@@ -3,11 +3,12 @@
   <xacro:include filename="$(find avatar_gripper_description)/urdf/avatar_gripper_3f_macro.xacro" />
   <xacro:avatar_gripper_3f prefix="right"/>
-  <!-- <xacro:macro name="attach_gripper" params="connected_to:='' arm_id:='panda' rpy:='0 0 0' xyz:='0 0 0'">
+  <xacro:macro name="attach_gripper" params="connected_to:='' arm_id='panda' gripper_prefix:='' rpy:='0 0 0' xyz:='0 0 0'">
     <xacro:unless value="${connected_to == ''}">
       <joint name="${arm_id}_gripper_joint" type="fixed">
         <parent link="${connected_to}" />
-        <child link="${arm_id}_hand" />
+        <child link="${gripper_prefix}_gripper_base" />
         <origin xyz="${xyz}" rpy="${rpy}" />
       </joint>
-    </xacro:unless>     -->
+    </xacro:unless>
+  </xacro:macro>
 </robot>
