Commit message: Expanded to dual arm model.

File: avatar_gripper_description/urdf/avatar_gripper_3f.xacro (robot description, xacro)
@@ -7,5 +7,4 @@
     <xacro:include filename="$(find avatar_gripper_description)/urdf/avatar_gripper_3f_macro_nomimic.xacro" />
   </xacro:unless>
-  <xacro:avatar_gripper_3f prefix="right"/>
   <xacro:macro name="attach_gripper" params="connected_to:='' arm_id='panda' gripper_prefix:='' rpy:='0 0 0' xyz:='0 0 0'">
     <xacro:unless value="${connected_to == ''}">

File: avatar_gripper_description/urdf/avatar_gripper_3f_macro.xacro (robot description, xacro)
@@ -10,5 +10,5 @@
         <origin xyz="0 0 0" rpy="0 0 0"/>
         <geometry>
-          <mesh filename="package://avatar_gripper_description/meshes/gripper_base.obj"/>
+          <mesh filename="package://avatar_gripper_description/meshes/${prefix}/gripper_base.obj"/>
         </geometry>
         <material name="">
@@ -27,14 +27,14 @@
         <origin xyz="0 0 0" rpy="0 0 0"/>
         <geometry>
-          <mesh filename="package://avatar_gripper_description/meshes/thumb_base_extra.obj"/>
-        </geometry>
-        <material name="">
-          <color rgba="0.9 0.9 0.9 1"/>
-        </material>
-      </visual>
-      <collision>
-        <origin xyz="0 0 0" rpy="0 0 0"/>
-        <geometry>
-          <mesh filename="package://avatar_gripper_description/meshes/thumb_base_extra.obj"/>
+          <mesh filename="package://avatar_gripper_description/meshes/${prefix}/thumb_base_extra.obj"/>
+        </geometry>
+        <material name="">
+          <color rgba="0.9 0.9 0.9 1"/>
+        </material>
+      </visual>
+      <collision>
+        <origin xyz="0 0 0" rpy="0 0 0"/>
+        <geometry>
+          <mesh filename="package://avatar_gripper_description/meshes/${prefix}/thumb_base_extra.obj"/>
         </geometry>
       </collision>
@@ -50,14 +50,14 @@
         <origin xyz="0 0 0" rpy="0 0 0"/>
         <geometry>
-          <mesh filename="package://avatar_gripper_description/meshes/thumb_knuckle.obj"/>
-        </geometry>
-        <material name="">
-          <color rgba="0.9 0.9 0.9 1"/>
-        </material>
-      </visual>
-      <collision>
-        <origin xyz="0 0 0" rpy="0 0 0"/>
-        <geometry>
-          <mesh filename="package://avatar_gripper_description/meshes/thumb_knuckle.obj"/>
+          <mesh filename="package://avatar_gripper_description/meshes/${prefix}/thumb_knuckle.obj"/>
+        </geometry>
+        <material name="">
+          <color rgba="0.9 0.9 0.9 1"/>
+        </material>
+      </visual>
+      <collision>
+        <origin xyz="0 0 0" rpy="0 0 0"/>
+        <geometry>
+          <mesh filename="package://avatar_gripper_description/meshes/${prefix}/thumb_knuckle.obj"/>
         </geometry>
       </collision>
@@ -73,14 +73,14 @@
         <origin xyz="0 0 0" rpy="0 0 0"/>
         <geometry>
-          <mesh filename="package://avatar_gripper_description/meshes/thumb_fingertip.obj"/>
-        </geometry>
-        <material name="">
-          <color rgba="0.9 0.9 0.9 1"/>
-        </material>
-      </visual>
-      <collision>
-        <origin xyz="0 0 0" rpy="0 0 0"/>
-        <geometry>
-          <mesh filename="package://avatar_gripper_description/meshes/thumb_fingertip.obj"/>
+          <mesh filename="package://avatar_gripper_description/meshes/${prefix}/thumb_fingertip.obj"/>
+        </geometry>
+        <material name="">
+          <color rgba="0.9 0.9 0.9 1"/>
+        </material>
+      </visual>
+      <collision>
+        <origin xyz="0 0 0" rpy="0 0 0"/>
+        <geometry>
+          <mesh filename="package://avatar_gripper_description/meshes/${prefix}/thumb_fingertip.obj"/>
         </geometry>
       </collision>
@@ -92,5 +92,5 @@
         <origin xyz="0 0 0" rpy="0 0 0"/>
         <geometry>
-          <mesh filename="package://avatar_gripper_description/meshes/index_base_connector.obj"/>
+          <mesh filename="package://avatar_gripper_description/meshes/${prefix}/index_base_connector.obj"/>
         </geometry>
         <material name="">
@@ -109,14 +109,14 @@
         <origin xyz="0 0 0" rpy="0 0 0"/>
         <geometry>
-          <mesh filename="package://avatar_gripper_description/meshes/index_knuckle.obj"/>
-        </geometry>
-        <material name="">
-          <color rgba="0.9 0.9 0.9 1"/>
-        </material>
-      </visual>
-      <collision>
-        <origin xyz="0 0 0" rpy="0 0 0"/>
-        <geometry>
-          <mesh filename="package://avatar_gripper_description/meshes/index_knuckle.obj"/>
+          <mesh filename="package://avatar_gripper_description/meshes/${prefix}/index_knuckle.obj"/>
+        </geometry>
+        <material name="">
+          <color rgba="0.9 0.9 0.9 1"/>
+        </material>
+      </visual>
+      <collision>
+        <origin xyz="0 0 0" rpy="0 0 0"/>
+        <geometry>
+          <mesh filename="package://avatar_gripper_description/meshes/${prefix}/index_knuckle.obj"/>
         </geometry>
       </collision>
@@ -132,14 +132,14 @@
         <origin xyz="0 0 0" rpy="0 0 0"/>
         <geometry>
-          <mesh filename="package://avatar_gripper_description/meshes/index_fingertip.obj"/>
-        </geometry>
-        <material name="">
-          <color rgba="0.9 0.9 0.9 1"/>
-        </material>
-      </visual>
-      <collision>
-        <origin xyz="0 0 0" rpy="0 0 0"/>
-        <geometry>
-          <mesh filename="package://avatar_gripper_description/meshes/index_fingertip.obj"/>
+          <mesh filename="package://avatar_gripper_description/meshes/${prefix}/index_fingertip.obj"/>
+        </geometry>
+        <material name="">
+          <color rgba="0.9 0.9 0.9 1"/>
+        </material>
+      </visual>
+      <collision>
+        <origin xyz="0 0 0" rpy="0 0 0"/>
+        <geometry>
+          <mesh filename="package://avatar_gripper_description/meshes/${prefix}/index_fingertip.obj"/>
         </geometry>
       </collision>
@@ -155,14 +155,14 @@
         <origin xyz="0 0 0" rpy="0 0 0"/>
         <geometry>
-          <mesh filename="package://avatar_gripper_description/meshes/index_knuckle.obj"/>
-        </geometry>
-        <material name="">
-          <color rgba="0.9 0.9 0.9 1"/>
-        </material>
-      </visual>
-      <collision>
-        <origin xyz="0 0 0" rpy="0 0 0"/>
-        <geometry>
-          <mesh filename="package://avatar_gripper_description/meshes/index_knuckle.obj"/>
+          <mesh filename="package://avatar_gripper_description/meshes/${prefix}/index_knuckle.obj"/>
+        </geometry>
+        <material name="">
+          <color rgba="0.9 0.9 0.9 1"/>
+        </material>
+      </visual>
+      <collision>
+        <origin xyz="0 0 0" rpy="0 0 0"/>
+        <geometry>
+          <mesh filename="package://avatar_gripper_description/meshes/${prefix}/index_knuckle.obj"/>
         </geometry>
       </collision>
@@ -178,14 +178,14 @@
         <origin xyz="0 0 0" rpy="0 0 0"/>
         <geometry>
-          <mesh filename="package://avatar_gripper_description/meshes/index_fingertip.obj"/>
-        </geometry>
-        <material name="">
-          <color rgba="0.9 0.9 0.9 1"/>
-        </material>
-      </visual>
-      <collision>
-        <origin xyz="0 0 0" rpy="0 0 0"/>
-        <geometry>
-          <mesh filename="package://avatar_gripper_description/meshes/index_fingertip.obj"/>
+          <mesh filename="package://avatar_gripper_description/meshes/${prefix}/index_fingertip.obj"/>
+        </geometry>
+        <material name="">
+          <color rgba="0.9 0.9 0.9 1"/>
+        </material>
+      </visual>
+      <collision>
+        <origin xyz="0 0 0" rpy="0 0 0"/>
+        <geometry>
+          <mesh filename="package://avatar_gripper_description/meshes/${prefix}/index_fingertip.obj"/>
         </geometry>
       </collision>
@@ -197,5 +197,5 @@
         <origin xyz="0 0 0" rpy="0 0 0"/>
         <geometry>
-          <mesh filename="package://avatar_gripper_description/meshes/thumb_swivel_link.obj"/>
+          <mesh filename="package://avatar_gripper_description/meshes/${prefix}/thumb_swivel_link.obj"/>
         </geometry>
         <material name="">
@@ -235,5 +235,10 @@
   <xacro:macro name="thumb_swivel_joint" params="prefix">
     <joint name="${prefix}_thumb_swivel_joint" type="revolute">
-      <origin xyz="0 0 0.0173" rpy="0 0 0"/>
+      <xacro:if value="${prefix == 'left'}">
+        <origin xyz="0 0 0.0173" rpy="0 0 0.7853"/>
+      </xacro:if>
+      <xacro:if value="${prefix == 'right'}">
+        <origin xyz="0 0 0.0173" rpy="0 0 0"/>
+      </xacro:if>
       <parent link="${prefix}_index_base_connector"/>
       <child link="${prefix}_thumb_swivel_link"/>
@@ -245,5 +250,10 @@
   <xacro:macro name="index_knuckle_joint" params="prefix">
     <joint name="${prefix}_index_knuckle_joint" type="revolute">
-      <origin xyz="-0.021564878 0.008545 -0.0024358" rpy="1.94428593 1.07478656 1.98996937"/>
+      <xacro:if value="${prefix == 'left'}">
+        <origin xyz="+0.021564878 0.008545 -0.0024358" rpy="1.19730672 1.07478656 1.15162329"/>
+      </xacro:if>
+      <xacro:if value="${prefix == 'right'}">
+        <origin xyz="-0.021564878 0.008545 -0.0024358" rpy="1.94428593 1.07478656 1.98996937"/>
+      </xacro:if>
       <parent link="${prefix}_index_base_connector"/>
       <child link="${prefix}_index_knuckle"/>
@@ -265,5 +275,10 @@
   <xacro:macro name="middle_knuckle_joint" params="prefix">
     <joint name="${prefix}_middle_knuckle_joint" type="revolute">
-      <origin xyz="0.02156 0.008545 -0.0024358" rpy="1.19730672 1.07478656 1.15162329"/>
+      <xacro:if value="${prefix == 'left'}">
+        <origin xyz="-0.02156 0.008545 -0.0024358" rpy="1.94428593 1.07478656 1.98996937"/>
+      </xacro:if>
+      <xacro:if value="${prefix == 'right'}">
+        <origin xyz="0.02156 0.008545 -0.0024358" rpy="1.19730672 1.07478656 1.15162329"/>
+      </xacro:if>
       <parent link="${prefix}_index_base_connector"/>
       <child link="${prefix}_middle_knuckle"/>
@@ -285,5 +300,10 @@
   <xacro:macro name="gripper_base_joint" params="prefix">
     <joint name="${prefix}_gripper_base_joint" type="fixed">
-      <origin xyz="0.00736 0.139 -0.066017" rpy="1.57 0 0"/>
+      <xacro:if value="${prefix == 'left'}">
+        <origin xyz="-0.00736 0.139 -0.066017" rpy="1.57 0 0"/>
+      </xacro:if>
+      <xacro:if value="${prefix == 'right'}">
+        <origin xyz="0.00736 0.139 -0.066017" rpy="1.57 0 0"/>
+      </xacro:if>
       <parent link="${prefix}_gripper_base"/>
       <child link="${prefix}_index_base_connector"/>

File: avatar_gripper_description/urdf/avatar_gripper_3f_macro_nomimic.xacro (robot description, xacro)
@@ -10,5 +10,5 @@
         <origin xyz="0 0 0" rpy="0 0 0"/>
         <geometry>
-          <mesh filename="package://avatar_gripper_description/meshes/gripper_base.obj"/>
+          <mesh filename="package://avatar_gripper_description/meshes/${prefix}/gripper_base.obj"/>
         </geometry>
         <material name="">
@@ -27,14 +27,14 @@
         <origin xyz="0 0 0" rpy="0 0 0"/>
         <geometry>
-          <mesh filename="package://avatar_gripper_description/meshes/thumb_base_extra.obj"/>
-        </geometry>
-        <material name="">
-          <color rgba="0.9 0.9 0.9 1"/>
-        </material>
-      </visual>
-      <collision>
-        <origin xyz="0 0 0" rpy="0 0 0"/>
-        <geometry>
-          <mesh filename="package://avatar_gripper_description/meshes/thumb_base_extra.obj"/>
+          <mesh filename="package://avatar_gripper_description/meshes/${prefix}/thumb_base_extra.obj"/>
+        </geometry>
+        <material name="">
+          <color rgba="0.9 0.9 0.9 1"/>
+        </material>
+      </visual>
+      <collision>
+        <origin xyz="0 0 0" rpy="0 0 0"/>
+        <geometry>
+          <mesh filename="package://avatar_gripper_description/meshes/${prefix}/thumb_base_extra.obj"/>
         </geometry>
       </collision>
@@ -50,14 +50,14 @@
         <origin xyz="0 0 0" rpy="0 0 0"/>
         <geometry>
-          <mesh filename="package://avatar_gripper_description/meshes/thumb_knuckle.obj"/>
-        </geometry>
-        <material name="">
-          <color rgba="0.9 0.9 0.9 1"/>
-        </material>
-      </visual>
-      <collision>
-        <origin xyz="0 0 0" rpy="0 0 0"/>
-        <geometry>
-          <mesh filename="package://avatar_gripper_description/meshes/thumb_knuckle.obj"/>
+          <mesh filename="package://avatar_gripper_description/meshes/${prefix}/thumb_knuckle.obj"/>
+        </geometry>
+        <material name="">
+          <color rgba="0.9 0.9 0.9 1"/>
+        </material>
+      </visual>
+      <collision>
+        <origin xyz="0 0 0" rpy="0 0 0"/>
+        <geometry>
+          <mesh filename="package://avatar_gripper_description/meshes/${prefix}/thumb_knuckle.obj"/>
         </geometry>
       </collision>
@@ -73,14 +73,14 @@
         <origin xyz="0 0 0" rpy="0 0 0"/>
         <geometry>
-          <mesh filename="package://avatar_gripper_description/meshes/thumb_fingertip.obj"/>
-        </geometry>
-        <material name="">
-          <color rgba="0.9 0.9 0.9 1"/>
-        </material>
-      </visual>
-      <collision>
-        <origin xyz="0 0 0" rpy="0 0 0"/>
-        <geometry>
-          <mesh filename="package://avatar_gripper_description/meshes/thumb_fingertip.obj"/>
+          <mesh filename="package://avatar_gripper_description/meshes/${prefix}/thumb_fingertip.obj"/>
+        </geometry>
+        <material name="">
+          <color rgba="0.9 0.9 0.9 1"/>
+        </material>
+      </visual>
+      <collision>
+        <origin xyz="0 0 0" rpy="0 0 0"/>
+        <geometry>
+          <mesh filename="package://avatar_gripper_description/meshes/${prefix}/thumb_fingertip.obj"/>
         </geometry>
       </collision>
@@ -92,5 +92,5 @@
         <origin xyz="0 0 0" rpy="0 0 0"/>
         <geometry>
-          <mesh filename="package://avatar_gripper_description/meshes/index_base_connector.obj"/>
+          <mesh filename="package://avatar_gripper_description/meshes/${prefix}/index_base_connector.obj"/>
         </geometry>
         <material name="">
@@ -109,14 +109,14 @@
         <origin xyz="0 0 0" rpy="0 0 0"/>
         <geometry>
-          <mesh filename="package://avatar_gripper_description/meshes/index_knuckle.obj"/>
-        </geometry>
-        <material name="">
-          <color rgba="0.9 0.9 0.9 1"/>
-        </material>
-      </visual>
-      <collision>
-        <origin xyz="0 0 0" rpy="0 0 0"/>
-        <geometry>
-          <mesh filename="package://avatar_gripper_description/meshes/index_knuckle.obj"/>
+          <mesh filename="package://avatar_gripper_description/meshes/${prefix}/index_knuckle.obj"/>
+        </geometry>
+        <material name="">
+          <color rgba="0.9 0.9 0.9 1"/>
+        </material>
+      </visual>
+      <collision>
+        <origin xyz="0 0 0" rpy="0 0 0"/>
+        <geometry>
+          <mesh filename="package://avatar_gripper_description/meshes/${prefix}/index_knuckle.obj"/>
         </geometry>
       </collision>
@@ -132,14 +132,14 @@
         <origin xyz="0 0 0" rpy="0 0 0"/>
         <geometry>
-          <mesh filename="package://avatar_gripper_description/meshes/index_fingertip.obj"/>
-        </geometry>
-        <material name="">
-          <color rgba="0.9 0.9 0.9 1"/>
-        </material>
-      </visual>
-      <collision>
-        <origin xyz="0 0 0" rpy="0 0 0"/>
-        <geometry>
-          <mesh filename="package://avatar_gripper_description/meshes/index_fingertip.obj"/>
+          <mesh filename="package://avatar_gripper_description/meshes/${prefix}/index_fingertip.obj"/>
+        </geometry>
+        <material name="">
+          <color rgba="0.9 0.9 0.9 1"/>
+        </material>
+      </visual>
+      <collision>
+        <origin xyz="0 0 0" rpy="0 0 0"/>
+        <geometry>
+          <mesh filename="package://avatar_gripper_description/meshes/${prefix}/index_fingertip.obj"/>
         </geometry>
       </collision>
@@ -155,14 +155,14 @@
         <origin xyz="0 0 0" rpy="0 0 0"/>
         <geometry>
-          <mesh filename="package://avatar_gripper_description/meshes/index_knuckle.obj"/>
-        </geometry>
-        <material name="">
-          <color rgba="0.9 0.9 0.9 1"/>
-        </material>
-      </visual>
-      <collision>
-        <origin xyz="0 0 0" rpy="0 0 0"/>
-        <geometry>
-          <mesh filename="package://avatar_gripper_description/meshes/index_knuckle.obj"/>
+          <mesh filename="package://avatar_gripper_description/meshes/${prefix}/index_knuckle.obj"/>
+        </geometry>
+        <material name="">
+          <color rgba="0.9 0.9 0.9 1"/>
+        </material>
+      </visual>
+      <collision>
+        <origin xyz="0 0 0" rpy="0 0 0"/>
+        <geometry>
+          <mesh filename="package://avatar_gripper_description/meshes/${prefix}/index_knuckle.obj"/>
         </geometry>
       </collision>
@@ -178,15 +178,12 @@
         <origin xyz="0 0 0" rpy="0 0 0"/>
         <geometry>
-          <mesh filename="package://avatar_gripper_description/meshes/index_fingertip.obj"/>
-        </geometry>
-        <material name="">
-          <color rgba="0.9 0.9 0.9 1"/>
-        </material>
-      </visual>
-      <collision>
-        <origin xyz="0 0 0" rpy="0 0 0"/>
-        <geometry>
-          <mesh filename="package://avatar_gripper_description/meshes/index_fingertip.obj"/>
-        </geometry>
+          <mesh filename="package://avatar_gripper_description/meshes/${prefix}/index_fingertip.obj"/>
+        </geometry>
+        <material name="">
+          <color rgba="0.9 0.9 0.9 1"/>
+        </material>
+      </visual>
+      <collision>
+        <origin xyz="0 0 0" rpy="0 0 0"/>
       </collision>
     </link>
@@ -197,5 +194,5 @@
         <origin xyz="0 0 0" rpy="0 0 0"/>
         <geometry>
-          <mesh filename="package://avatar_gripper_description/meshes/thumb_swivel_link.obj"/>
+          <mesh filename="package://avatar_gripper_description/meshes/${prefix}/thumb_swivel_link.obj"/>
         </geometry>
         <material name="">
@@ -233,5 +230,10 @@
   <xacro:macro name="thumb_swivel_joint" params="prefix">
     <joint name="${prefix}_thumb_swivel_joint" type="revolute">
-      <origin xyz="0 0 0.0173" rpy="0 0 0"/>
+      <xacro:if value="${prefix == 'left'}">
+        <origin xyz="0 0 0.0173" rpy="0 0 0.7853"/>
+      </xacro:if>
+      <xacro:if value="${prefix == 'right'}">
+        <origin xyz="0 0 0.0173" rpy="0 0 0"/>
+      </xacro:if>
       <parent link="${prefix}_index_base_connector"/>
       <child link="${prefix}_thumb_swivel_link"/>
@@ -242,5 +244,10 @@
   <xacro:macro name="index_knuckle_joint" params="prefix">
     <joint name="${prefix}_index_knuckle_joint" type="revolute">
-      <origin xyz="-0.021564878 0.008545 -0.0024358" rpy="1.94428593 1.07478656 1.98996937"/>
+      <xacro:if value="${prefix == 'left'}">
+        <origin xyz="+0.021564878 0.008545 -0.0024358" rpy="1.19730672 1.07478656 1.15162329"/>
+      </xacro:if>
+      <xacro:if value="${prefix == 'right'}">
+        <origin xyz="-0.021564878 0.008545 -0.0024358" rpy="1.94428593 1.07478656 1.98996937"/>
+      </xacro:if>
       <parent link="${prefix}_index_base_connector"/>
       <child link="${prefix}_index_knuckle"/>
@@ -260,5 +267,10 @@
   <xacro:macro name="middle_knuckle_joint" params="prefix">
     <joint name="${prefix}_middle_knuckle_joint" type="revolute">
-      <origin xyz="0.02156 0.008545 -0.0024358" rpy="1.19730672 1.07478656 1.15162329"/>
+      <xacro:if value="${prefix == 'left'}">
+        <origin xyz="-0.02156 0.008545 -0.0024358" rpy="1.94428593 1.07478656 1.98996937"/>
+      </xacro:if>
+      <xacro:if value="${prefix == 'right'}">
+        <origin xyz="0.02156 0.008545 -0.0024358" rpy="1.19730672 1.07478656 1.15162329"/>
+      </xacro:if>
       <parent link="${prefix}_index_base_connector"/>
       <child link="${prefix}_middle_knuckle"/>
@@ -278,5 +290,10 @@
   <xacro:macro name="gripper_base_joint" params="prefix">
     <joint name="${prefix}_gripper_base_joint" type="fixed">
-      <origin xyz="0.00736 0.139 -0.066017" rpy="1.57 0 0"/>
+      <xacro:if value="${prefix == 'left'}">
+        <origin xyz="-0.00736 0.139 -0.066017" rpy="1.57 0 0"/>
+      </xacro:if>
+      <xacro:if value="${prefix == 'right'}">
+        <origin xyz="0.00736 0.139 -0.066017" rpy="1.57 0 0"/>
+      </xacro:if>
       <parent link="${prefix}_gripper_base"/>
       <child link="${prefix}_index_base_connector"/>

File: avatar_robot_description/franka/common/franka_arm.xacro (robot description, xacro)
@@ -13,5 +13,5 @@
       </joint>
     </xacro:unless>
-    <xacro:link_with_sc name="link0" gazebo="${gazebo}">
+    <xacro:link_with_sc name="link0" gazebo="${gazebo}" rpy='0 0 0'>
       <self_collision_geometries>
         <xacro:collision_capsule xyz="-0.075 0 0.06" direction="x" radius="${0.06+safety_distance}" length="0.03" />

File: avatar_robot_description/franka/common/franka_robot.xacro (robot description, xacro)
@@ -22,5 +22,5 @@
           rpy="0 ${pi} ${-pi/4}"
           connected_to="$(arg arm_id)_link8"
-          gripper_prefix="right"
+          gripper_prefix="left"
        />
     </xacro:if>

File: avatar_robot_description/franka/common/hand.urdf.xacro (robot description, xacro)
@@ -2,5 +2,10 @@
 <robot xmlns:xacro="http://www.ros.org/wiki/xacro" name="hand">
   <xacro:include filename="$(find franka_description)/robots/common/utils.xacro" />
+  <xacro:if value="$(prefix)=='right'">
+    <xacro:franka_hand arm_id="panda_1" safety_distance="0.03"/>
+  </xacro:if>
   <xacro:include filename="franka_hand.xacro"/>
-  <xacro:franka_hand arm_id="panda" safety_distance="0.03"/>
+  <xacro:if value="$(prefix)=='left'">
+    <xacro:franka_hand arm_id="panda_2" safety_distance="0.03"/>
+  </xacro:if>
 </robot>
