Commit message: Expanded to dual arm model.

File: avatar_robot_description/franka/dual_panda/dual_panda_example.urdf.xacro (robot description, xacro)
@@ -1,31 +1,18 @@
 <?xml version="1.0" encoding="utf-8"?>
 <robot xmlns:xacro="http://www.ros.org/wiki/xacro" name="panda">
-  <xacro:arg name="arm_id_1" default="panda_1" />
-  <xacro:arg name="arm_id_2" default="panda_2" />
-  <xacro:include filename="$(find franka_description)/robots/common/franka_arm.xacro"/>
-  <xacro:include filename="$(find franka_description)/robots/common/franka_hand.xacro"/>
-  <!-- box shaped table as base for the 2 Pandas -->
-  <link name="base">
-    <visual>
-      <origin xyz="0 0 0.5" rpy="0 0 0"/>
-      <geometry>
-        <box size="1 2 1" />
-      </geometry>
-      <material name="White">
-        <color rgba="1.0 1.0 1.0 1.0"/>
-      </material>
-    </visual>
-    <collision>
-      <origin xyz="0 0 0.5" rpy="0 0 0"/>
-      <geometry>
-        <box size="1 2 1" />
-      </geometry>
-    </collision>
-  </link>
+  <xacro:arg name="arm_id_1" default="right_panda" />
+  <xacro:arg name="arm_id_2" default="left_panda" />
+  <xacro:arg name="pref_1" default="right" />
+  <xacro:arg name="pref_2" default="left" />
+  <xacro:include filename="$(find avatar_robot_description)/franka/common/franka_arm.xacro"/>
+  <xacro:include filename="$(find avatar_robot_description)/franka/common/base.xacro"/>
+  <xacro:include filename="$(find avatar_gripper_description)/urdf/avatar_gripper_3f.xacro"/>
   <!-- right arm with gripper -->
-  <xacro:franka_arm arm_id="$(arg arm_id_1)" connected_to="base"  xyz="0 -0.5 1" safety_distance="0.03" joint_limits="${xacro.load_yaml('$(find franka_description)/robots/panda/joint_limits.yaml')}"/>
-  <xacro:franka_hand arm_id="$(arg arm_id_1)" rpy="0 0 ${-pi/4}" connected_to="$(arg arm_id_1)_link8" safety_distance="0.03"/>
+  <xacro:franka_arm arm_id="$(arg arm_id_1)" connected_to="support"  xyz="${length_support*0.45} ${-dist_arms/2} ${heigth_support/2}" rpy='0 0 0' safety_distance="0.03" joint_limits="${xacro.load_yaml('$(find avatar_robot_description)/franka/panda/joint_limits.yaml')}"/>
+  <xacro:avatar_gripper_3f prefix="$(arg pref_1)"/>
+  <xacro:attach_gripper connected_to="$(arg arm_id_1)_link8" arm_id="$(arg arm_id_1)" gripper_prefix='right' rpy="0 ${pi} ${-pi/4}" xyz='0 0 0'/>
   <!-- left arm with gripper -->
-  <xacro:franka_arm arm_id="$(arg arm_id_2)" connected_to="base"  xyz="0 0.5 1" safety_distance="0.03" joint_limits="${xacro.load_yaml('$(find franka_description)/robots/panda/joint_limits.yaml')}"/>
-  <xacro:franka_hand arm_id="$(arg arm_id_2)" rpy="0 0 ${-pi/4}" connected_to="$(arg arm_id_2)_link8" safety_distance="0.03"/>
+  <xacro:franka_arm arm_id="$(arg arm_id_2)" connected_to="support"  xyz="${length_support*0.45} ${dist_arms/2} ${heigth_support/2}" rpy='0 0 0' safety_distance="0.03" joint_limits="${xacro.load_yaml('$(find avatar_robot_description)/franka/panda/joint_limits.yaml')}"/>
+  <xacro:avatar_gripper_3f prefix="$(arg pref_2)"/>
+  <xacro:attach_gripper connected_to="$(arg arm_id_2)_link8" arm_id="$(arg arm_id_2)" gripper_prefix='left' rpy="0 ${pi} ${-pi/4}" xyz='0 0 0'/>
 </robot>

File: avatar_robot_description/urdf/panda_with_gripper.urdf (robot description, URDF)
Before this commit: robot panda, 30 links, 29 joints
Links:
- removed link right_gripper_base
- removed link right_index_base_connector
- removed link right_index_fingertip
- removed link right_index_flex_motor
- removed link right_index_knuckle
- removed link right_middle_fingertip
- removed link right_middle_knuckle
- removed link right_thumb_base
- removed link right_thumb_finger
- removed link right_thumb_flex_motor
- removed link right_thumb_knuckle
- removed link right_thumb_swivel_link
- removed link right_thumb_swivel_motor
- added link left_gripper_base, mass 2.0; visual mesh filename=package://avatar_gripper_description/meshes/gripper_base.obj
- added link left_index_base_connector; visual mesh filename=package://avatar_gripper_description/meshes/index_base_conn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
- added link left_index_fingertip, mass 0.5; collision mesh filename=package://avatar_gripper_description/meshes/index_fingertip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; visual mesh filename=package://avatar_gripper_description/meshes/index_fingertip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
- added link left_index_flex_motor, mass 0.25; visual cylinder length=0.01 radius=0.02
- added link left_index_knuckle, mass 0.5; collision mesh filename=package://avatar_gripper_description/meshes/index_knuckle.o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; visual mesh filename=package://avatar_gripper_description/meshes/index_knuckle.o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
- added link left_middle_fingertip, mass 0.5; collision mesh filename=package://avatar_gripper_description/meshes/index_fingertip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; visual mesh filename=package://avatar_gripper_description/meshes/index_fingertip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
- added link left_middle_knuckle, mass 0.5; collision mesh filename=package://avatar_gripper_description/meshes/index_knuckle.o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; visual mesh filename=package://avatar_gripper_description/meshes/index_knuckle.o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
- added link left_thumb_base, mass 0.5; collision mesh filename=package://avatar_gripper_description/meshes/thumb_base_extr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; visual mesh filename=package://avatar_gripper_description/meshes/thumb_base_extr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
- added link left_thumb_finger, mass 0.5; collision mesh filename=package://avatar_gripper_description/meshes/thumb_fingertip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; visual mesh filename=package://avatar_gripper_description/meshes/thumb_fingertip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
- added link left_thumb_flex_motor, mass 0.25; visual cylinder length=0.01 radius=0.02
- added link left_thumb_knuckle, mass 0.5; collision mesh filename=package://avatar_gripper_description/meshes/thumb_knuckle.o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; visual mesh filename=package://avatar_gripper_description/meshes/thumb_knuckle.o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
- added link left_thumb_swivel_link; visual mesh filename=package://avatar_gripper_description/meshes/thumb_swivel_li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
- added link left_thumb_swivel_motor, mass 0.25; visual cylinder length=0.01 radius=0.02
Joints:
- removed joint right_gripper_base_joint
- removed joint right_index_fingertip_joint
- removed joint right_index_flex_motor_joint
- removed joint right_index_knuckle_joint
- removed joint right_middle_fingertip_joint
- removed joint right_middle_knuckle_joint
- removed joint right_thumb_base_swivel_joint
- removed joint right_thumb_finger_joint
- removed joint right_thumb_flex_motor_joint
- removed joint right_thumb_knuckle_joint
- removed joint right_thumb_swivel_joint
- removed joint right_thumb_swivel_motor_joint
- added joint left_gripper_base_joint: type fixed, parent left_gripper_base, child left_index_base_connector, origin xyz=0.00736 0.139 -0.066017 rpy=1.57 0 0
- added joint left_index_fingertip_joint: type revolute, parent left_index_knuckle, child left_index_fingertip, origin xyz=0.0353829 -0.02780 0 rpy=0 0 -0.35, axis 0 0 1, limit lower=-0.8 upper=0 effort=1000 velocity=2.0, mimic joint=left_index_flex_motor_joint multiplier=0.4 offset=0
- added joint left_index_flex_motor_joint: type revolute, parent left_gripper_base, child left_index_flex_motor, origin xyz=0 -0.3 0 rpy=0 0 0, axis 0 0 1, limit lower=-2.3 upper=-0.08 effort=1000 velocity=2.0
- added joint left_index_knuckle_joint: type revolute, parent left_index_base_connector, child left_index_knuckle, origin xyz=-0.021564878 0.008545 -0.0024358 rpy=1.94428593 1.07478656 1.98996937, axis 0 0 1, limit lower=-0.8 upper=0 effort=1000 velocity=2.0, mimic joint=left_index_flex_motor_joint multiplier=0.4016 offset=0
- added joint left_middle_fingertip_joint: type revolute, parent left_middle_knuckle, child left_middle_fingertip, origin xyz=0.0353829 -0.02780 0 rpy=0 0 -0.35, axis 0 0 1, limit lower=-0.8 upper=0 effort=1000 velocity=2.0, mimic joint=left_index_fingertip_joint multiplier=1 offset=0
- added joint left_middle_knuckle_joint: type revolute, parent left_index_base_connector, child left_middle_knuckle, origin xyz=0.02156 0.008545 -0.0024358 rpy=1.19730672 1.07478656 1.15162329, axis 0 0 1, limit lower=-0.8 upper=0 effort=1000 velocity=2.0, mimic joint=left_index_knuckle_joint multiplier=1 offset=0
- added joint left_thumb_base_swivel_joint: type fixed, parent left_thumb_swivel_link, child left_thumb_base, origin xyz=-0.03742 0 0.05089 rpy=0 0 0
- added joint left_thumb_finger_joint: type revolute, parent left_thumb_knuckle, child left_thumb_finger, origin xyz=0.04568 0 0.01106 rpy=0 0.57 0, axis 0 1 0, limit lower=-0.8 upper=0 effort=1000 velocity=2.0, mimic joint=left_thumb_flex_motor_joint multiplier=0.24 offset=0
- added joint left_thumb_flex_motor_joint: type revolute, parent left_gripper_base, child left_thumb_flex_motor, origin xyz=-0.05 -0.3 0 rpy=0 0 0, axis 0 0 1, limit lower=-2.3 upper=-0.08 effort=1000 velocity=2.0
- added joint left_thumb_knuckle_joint: type revolute, parent left_thumb_base, child left_thumb_knuckle, origin xyz=0 0 0 rpy=0 2.75 0, axis 0 1 0, limit lower=-1.0 upper=0.4 effort=1000 velocity=2.0, mimic joint=left_thumb_flex_motor_joint multiplier=0.28 offset=0
- added joint left_thumb_swivel_joint: type revolute, parent left_index_base_connector, child left_thumb_swivel_link, origin xyz=0 0 0.0173 rpy=0 0 0, axis 0 0 1, limit lower=0 upper=1.7 effort=1000 velocity=2.0, mimic joint=left_thumb_swivel_motor_joint multiplier=-0.6075 offset=0.43
- added joint left_thumb_swivel_motor_joint: type revolute, parent left_gripper_base, child left_thumb_swivel_motor, origin xyz=-0.1 -0.3 0 rpy=0 0 0, axis 0 0 1, limit lower=-2.3 upper=-0.05 effort=1000 velocity=2.0
- joint panda_gripper_joint: child right_gripper_base -> left_gripper_base

File: avatar_robot_description/urdf/panda_with_gripper_nomimic.urdf (robot description, URDF)
Before this commit: robot panda, 30 links, 29 joints
Links:
- removed link right_gripper_base
- removed link right_index_base_connector
- removed link right_index_fingertip
- removed link right_index_flex_motor
- removed link right_index_knuckle
- removed link right_middle_fingertip
- removed link right_middle_knuckle
- removed link right_thumb_base
- removed link right_thumb_finger
- removed link right_thumb_flex_motor
- removed link right_thumb_knuckle
- removed link right_thumb_swivel_link
- removed link right_thumb_swivel_motor
- added link left_gripper_base, mass 2.0; visual mesh filename=package://avatar_gripper_description/meshes/gripper_base.obj
- added link left_index_base_connector; visual mesh filename=package://avatar_gripper_description/meshes/index_base_conn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
- added link left_index_fingertip, mass 0.5; collision mesh filename=package://avatar_gripper_description/meshes/index_fingertip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; visual mesh filename=package://avatar_gripper_description/meshes/index_fingertip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
- added link left_index_flex_motor, mass 0.25; visual cylinder length=0.01 radius=0.02
- added link left_index_knuckle, mass 0.5; collision mesh filename=package://avatar_gripper_description/meshes/index_knuckle.o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; visual mesh filename=package://avatar_gripper_description/meshes/index_knuckle.o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
- added link left_middle_fingertip, mass 0.5; collision mesh filename=package://avatar_gripper_description/meshes/index_fingertip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; visual mesh filename=package://avatar_gripper_description/meshes/index_fingertip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
- added link left_middle_knuckle, mass 0.5; collision mesh filename=package://avatar_gripper_description/meshes/index_knuckle.o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; visual mesh filename=package://avatar_gripper_description/meshes/index_knuckle.o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
- added link left_thumb_base, mass 0.5; collision mesh filename=package://avatar_gripper_description/meshes/thumb_base_extr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; visual mesh filename=package://avatar_gripper_description/meshes/thumb_base_extr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
- added link left_thumb_finger, mass 0.5; collision mesh filename=package://avatar_gripper_description/meshes/thumb_fingertip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; visual mesh filename=package://avatar_gripper_description/meshes/thumb_fingertip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
- added link left_thumb_flex_motor, mass 0.25; visual cylinder length=0.01 radius=0.02
- added link left_thumb_knuckle, mass 0.5; collision mesh filename=package://avatar_gripper_description/meshes/thumb_knuckle.o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; visual mesh filename=package://avatar_gripper_description/meshes/thumb_knuckle.o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
- added link left_thumb_swivel_link; visual mesh filename=package://avatar_gripper_description/meshes/thumb_swivel_li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
- added link left_thumb_swivel_motor, mass 0.25; visual cylinder length=0.01 radius=0.02
Joints:
- removed joint right_gripper_base_joint
- removed joint right_index_fingertip_joint
- removed joint right_index_flex_motor_joint
- removed joint right_index_knuckle_joint
- removed joint right_middle_fingertip_joint
- removed joint right_middle_knuckle_joint
- removed joint right_thumb_base_swivel_joint
- removed joint right_thumb_finger_joint
- removed joint right_thumb_flex_motor_joint
- removed joint right_thumb_knuckle_joint
- removed joint right_thumb_swivel_joint
- removed joint right_thumb_swivel_motor_joint
- added joint left_gripper_base_joint: type fixed, parent left_gripper_base, child left_index_base_connector, origin xyz=0.00736 0.139 -0.066017 rpy=1.57 0 0
- added joint left_index_fingertip_joint: type revolute, parent left_index_knuckle, child left_index_fingertip, origin xyz=0.0353829 -0.02780 0 rpy=0 0 -0.35, axis 0 0 1, limit lower=-0.8 upper=0 effort=1000 velocity=2.0
- added joint left_index_flex_motor_joint: type revolute, parent left_gripper_base, child left_index_flex_motor, origin xyz=0 -0.3 0 rpy=0 0 0, axis 0 0 1, limit lower=-2.3 upper=-0.08 effort=1000 velocity=2.0
- added joint left_index_knuckle_joint: type revolute, parent left_index_base_connector, child left_index_knuckle, origin xyz=-0.021564878 0.008545 -0.0024358 rpy=1.94428593 1.07478656 1.98996937, axis 0 0 1, limit lower=-0.8 upper=0 effort=1000 velocity=2.0
- added joint left_middle_fingertip_joint: type revolute, parent left_middle_knuckle, child left_middle_fingertip, origin xyz=0.0353829 -0.02780 0 rpy=0 0 -0.35, axis 0 0 1, limit lower=-0.8 upper=0 effort=1000 velocity=2.0
- added joint left_middle_knuckle_joint: type revolute, parent left_index_base_connector, child left_middle_knuckle, origin xyz=0.02156 0.008545 -0.0024358 rpy=1.19730672 1.07478656 1.15162329, axis 0 0 1, limit lower=-0.8 upper=0 effort=1000 velocity=2.0
- added joint left_thumb_base_swivel_joint: type fixed, parent left_thumb_swivel_link, child left_thumb_base, origin xyz=-0.03742 0 0.05089 rpy=0 0 0
- added joint left_thumb_finger_joint: type revolute, parent left_thumb_knuckle, child left_thumb_finger, origin xyz=0.04568 0 0.01106 rpy=0 0.57 0, axis 0 1 0, limit lower=-0.8 upper=0 effort=1000 velocity=2.0
- added joint left_thumb_flex_motor_joint: type revolute, parent left_gripper_base, child left_thumb_flex_motor, origin xyz=-0.05 -0.3 0 rpy=0 0 0, axis 0 0 1, limit lower=-2.3 upper=-0.08 effort=1000 velocity=2.0
- added joint left_thumb_knuckle_joint: type revolute, parent left_thumb_base, child left_thumb_knuckle, origin xyz=0 0 0 rpy=0 2.75 0, axis 0 1 0, limit lower=-1.0 upper=0.4 effort=1000 velocity=2.0
- added joint left_thumb_swivel_joint: type revolute, parent left_index_base_connector, child left_thumb_swivel_link, origin xyz=0 0 0.0173 rpy=0 0 0, axis 0 0 1, limit lower=0 upper=1.7 effort=1000 velocity=2.0
- added joint left_thumb_swivel_motor_joint: type revolute, parent left_gripper_base, child left_thumb_swivel_motor, origin xyz=-0.1 -0.3 0 rpy=0 0 0, axis 0 0 1, limit lower=-2.3 upper=-0.05 effort=1000 velocity=2.0
- joint panda_gripper_joint: child right_gripper_base -> left_gripper_base

Commit message: Simplified xacro implemetations for mimic/no-mimic behaviors Now the 3 gripper motors are fixed relative to the arm base_link when arm is available

File: avatar_gripper_description/urdf/avatar_gripper_3f.xacro (robot description, xacro)
@@ -1,10 +1,5 @@
 <?xml version="1.0"?>
 <robot name="avatar_gripper_3f_model" xmlns:xacro="http://ros.org/wiki/xacro">
-  <xacro:if value="$(arg mimic)">
-    <xacro:include filename="$(find avatar_gripper_description)/urdf/avatar_gripper_3f_macro.xacro" />
-  </xacro:if>
-  <xacro:unless value="$(arg mimic)">
-    <xacro:include filename="$(find avatar_gripper_description)/urdf/avatar_gripper_3f_macro_nomimic.xacro" />
-  </xacro:unless>
+  <xacro:include filename="$(find avatar_gripper_description)/urdf/avatar_gripper_3f_macro.xacro" />
   <xacro:macro name="attach_gripper" params="connected_to:='' arm_id='panda' gripper_prefix:='' rpy:='0 0 0' xyz:='0 0 0'">
     <xacro:unless value="${connected_to == ''}">

File: avatar_gripper_description/urdf/avatar_gripper_3f_example.xacro (robot description, xacro)
@@ -3,11 +3,7 @@
   <xacro:arg name="mimic" default="true"/>
   <xacro:arg name="prefix" default="right"/>
-  <xacro:if value="$(arg mimic)">
-    <xacro:include filename="$(find avatar_gripper_description)/urdf/avatar_gripper_3f_macro.xacro" />
-  </xacro:if>
-  <xacro:unless value="$(arg mimic)">
-    <xacro:include filename="$(find avatar_gripper_description)/urdf/avatar_gripper_3f_macro_nomimic.xacro" />
-  </xacro:unless>
-  <xacro:avatar_gripper_3f prefix="$(arg prefix)"/>
+  <xacro:arg name="motor_base_attach_to" default="right_gripper_base"/>
+  <xacro:include filename="$(find avatar_gripper_description)/urdf/avatar_gripper_3f_macro.xacro" />
+  <xacro:avatar_gripper_3f prefix="$(arg prefix)" motor_base_attach_to="$(arg motor_base_attach_to)"/>
   <xacro:macro name="attach_gripper" params="connected_to:='' arm_id='panda' gripper_prefix:='' rpy:='0 0 0' xyz:='0 0 0'">
     <xacro:unless value="${connected_to == ''}">

File: avatar_gripper_description/urdf/avatar_gripper_3f_macro.xacro (robot description, xacro)
@@ -233,5 +233,7 @@
       <axis xyz="0 1 0"/>
       <limit lower="-1.0" upper="0.4" velocity="2.0" effort="1000" />
-      <mimic joint="${prefix}_thumb_flex_motor_joint" offset="0" multiplier="0.28"/>
+      <xacro:if value="$(arg mimic)">
+        <mimic joint="${prefix}_thumb_flex_motor_joint" offset="0" multiplier="0.28"/>
+      </xacro:if>
     </joint>
   </xacro:macro>
@@ -243,5 +245,7 @@
       <axis xyz="0 1 0"/>
       <limit lower="-0.8" upper="0" velocity="2.0" effort="1000" />
-      <mimic joint="${prefix}_thumb_flex_motor_joint" offset="0" multiplier="0.24"/>
+      <xacro:if value="$(arg mimic)">
+        <mimic joint="${prefix}_thumb_flex_motor_joint" offset="0" multiplier="0.24"/>
+      </xacro:if>
     </joint>
   </xacro:macro>
@@ -265,5 +269,7 @@
       <axis xyz="0 0 1"/>
       <limit lower="0" upper="1.7" velocity="2.0" effort="1000" />
-      <mimic joint="${prefix}_thumb_swivel_motor_joint" offset="0.43" multiplier="-0.6075"/>
+      <xacro:if value="$(arg mimic)">
+        <mimic joint="${prefix}_thumb_swivel_motor_joint" offset="0.43" multiplier="-0.6075"/>
+      </xacro:if>
     </joint>
   </xacro:macro>
@@ -280,5 +286,7 @@
       <axis xyz="0 0 1"/>
       <limit lower="-0.8" upper="0" velocity="2.0" effort="1000" />
-      <mimic joint="${prefix}_index_flex_motor_joint" offset="0" multiplier="0.4016"/>
+      <xacro:if value="$(arg mimic)">
+        <mimic joint="${prefix}_index_flex_motor_joint" offset="0" multiplier="0.4016"/>
+      </xacro:if>
     </joint>
   </xacro:macro>
@@ -290,5 +298,7 @@
       <axis xyz="0 0 1"/>
       <limit lower="-0.8" upper="0" velocity="2.0" effort="1000" />
-      <mimic joint="${prefix}_index_flex_motor_joint" offset="0" multiplier="0.4"/>
+      <xacro:if value="$(arg mimic)">
+        <mimic joint="${prefix}_index_flex_motor_joint" offset="0" multiplier="0.4"/>
+      </xacro:if>
     </joint>
   </xacro:macro>
@@ -305,5 +315,7 @@
       <axis xyz="0 0 1"/>
       <limit lower="-0.8" upper="0" velocity="2.0" effort="1000" />
-      <mimic joint="${prefix}_index_knuckle_joint" offset="0" multiplier="1"/>
+      <xacro:if value="$(arg mimic)">
+        <mimic joint="${prefix}_index_knuckle_joint" offset="0" multiplier="1"/>
+      </xacro:if>
     </joint>
   </xacro:macro>
@@ -315,5 +327,7 @@
       <axis xyz="0 0 1"/>
       <limit lower="-0.8" upper="0" velocity="2.0" effort="1000" />
-      <mimic joint="${prefix}_index_fingertip_joint" offset="0" multiplier="1"/>
+      <xacro:if value="$(arg mimic)">
+        <mimic joint="${prefix}_index_fingertip_joint" offset="0" multiplier="1"/>
+      </xacro:if>
     </joint>
   </xacro:macro>
@@ -346,8 +360,8 @@
   </xacro:macro>
   <!-- actuator joints -->
-  <xacro:macro name="index_flex_motor_joint" params="prefix">
+  <xacro:macro name="index_flex_motor_joint" params="prefix motor_base_attach_to">
     <joint name="${prefix}_index_flex_motor_joint" type="revolute">
-      <origin xyz="0 -0.3 0" rpy="0 0 0"/>
-      <parent link="${prefix}_gripper_base"/>
+      <origin xyz="0.0 0.0 0.0" rpy="0 0 0"/>
+      <parent link="${motor_base_attach_to}"/>
       <child link="${prefix}_index_flex_motor"/>
       <axis xyz="0 0 1"/>
@@ -355,8 +369,8 @@
     </joint>
   </xacro:macro>
-  <xacro:macro name="thumb_flex_motor_joint" params="prefix">
+  <xacro:macro name="thumb_flex_motor_joint" params="prefix motor_base_attach_to">
     <joint name="${prefix}_thumb_flex_motor_joint" type="revolute">
-      <origin xyz="-0.05 -0.3 0" rpy="0 0 0"/>
-      <parent link="${prefix}_gripper_base"/>
+      <origin xyz="-0.05 0.0 0.0" rpy="0 0 0"/>
+      <parent link="${motor_base_attach_to}"/>
       <child link="${prefix}_thumb_flex_motor"/>
       <axis xyz="0 0 1"/>
@@ -364,8 +378,8 @@
     </joint>
   </xacro:macro>
-  <xacro:macro name="thumb_swivel_motor_joint" params="prefix">
+  <xacro:macro name="thumb_swivel_motor_joint" params="prefix motor_base_attach_to">
     <joint name="${prefix}_thumb_swivel_motor_joint" type="revolute">
-      <origin xyz="-0.1 -0.3 0" rpy="0 0 0"/>
-      <parent link="${prefix}_gripper_base"/>
+      <origin xyz="-0.1 0.0 0.0" rpy="0 0 0"/>
+      <parent link="${motor_base_attach_to}"/>
       <child link="${prefix}_thumb_swivel_motor"/>
       <axis xyz="0 0 1"/>
@@ -373,5 +387,5 @@
     </joint>
   </xacro:macro>
-  <xacro:macro name="avatar_gripper_3f" params="prefix">
+  <xacro:macro name="avatar_gripper_3f" params="prefix motor_base_attach_to">
     <xacro:thumb_base_link prefix="${prefix}"/>
     <xacro:thumb_knuckle_link prefix="${prefix}"/>
@@ -394,9 +408,9 @@
     <xacro:gripper_base_joint prefix="${prefix}"/>
     <xacro:motor_link prefix="${prefix}" actuation="thumb_flex"/>
-    <xacro:thumb_flex_motor_joint prefix="${prefix}"/>
+    <xacro:thumb_flex_motor_joint prefix="${prefix}" motor_base_attach_to="${motor_base_attach_to}"/>
     <xacro:motor_link prefix="${prefix}" actuation="thumb_swivel"/>
-    <xacro:thumb_swivel_motor_joint prefix="${prefix}"/>
+    <xacro:thumb_swivel_motor_joint prefix="${prefix}" motor_base_attach_to="${motor_base_attach_to}"/>
     <xacro:motor_link prefix="${prefix}" actuation="index_flex"/>
-    <xacro:index_flex_motor_joint prefix="${prefix}"/>
+    <xacro:index_flex_motor_joint prefix="${prefix}" motor_base_attach_to="${motor_base_attach_to}"/>
   </xacro:macro>
 </robot>
