Commit message: corrected package name

File: avatar_gripper_description/urdf/avatar_gripper_3f_macro.xacro (robot description, xacro)
@@ -213,5 +213,5 @@
       <axis xyz="0 1 0"/>
       <limit lower="-1.0" upper="0.4" velocity="2.0" effort="1000" />
-      <mimic joint="${prefix}_thumb_flex_motor_joint" offsite="0" multiplier="0.5702"/>
+      <mimic joint="${prefix}_thumb_flex_motor_joint" offsite="0" multiplier="0.28"/>
     </joint>
   </xacro:macro>
@@ -223,5 +223,5 @@
       <axis xyz="0 1 0"/>
       <limit lower="-0.8" upper="0" velocity="2.0" effort="1000" />
-      <mimic joint="${prefix}_thumb_flex_motor_joint" offsite="0" multiplier="0.6007"/>
+      <mimic joint="${prefix}_thumb_flex_motor_joint" offsite="0" multiplier="0.24"/>
     </joint>
   </xacro:macro>
@@ -250,5 +250,5 @@
       <axis xyz="0 0 1"/>
       <limit lower="-0.8" upper="0" velocity="2.0" effort="1000" />
-      <mimic joint="${prefix}_index_flex_motor_joint" offsite="0" multiplier="1"/>
+      <mimic joint="${prefix}_index_flex_motor_joint" offsite="0" multiplier="0.4016"/>
     </joint>
   </xacro:macro>
@@ -260,5 +260,5 @@
       <axis xyz="0 0 1"/>
       <limit lower="-0.8" upper="0" velocity="2.0" effort="1000" />
-      <mimic joint="${prefix}_index_flex_motor_joint" offsite="0" multiplier="0.40"/>
+      <mimic joint="${prefix}_index_flex_motor_joint" offsite="0" multiplier="0.6"/>
     </joint>
   </xacro:macro>
@@ -312,5 +312,5 @@
       <child link="${prefix}_index_flex_motor"/>
       <axis xyz="0 0 1"/>
-      <limit lower="-1.0" upper="0.0" velocity="2.0" effort="1000" />
+      <limit lower="-2.3" upper="-0.08" velocity="2.0" effort="1000" />
     </joint>
   </xacro:macro>
@@ -321,5 +321,5 @@
       <child link="${prefix}_thumb_flex_motor"/>
       <axis xyz="0 0 1"/>
-      <limit lower="-1.0" upper="0.0" velocity="2.0" effort="1000" />
+      <limit lower="-2.3" upper="-0.08" velocity="2.0" effort="1000" />
     </joint>
   </xacro:macro>
@@ -330,5 +330,5 @@
       <child link="${prefix}_thumb_swivel_motor"/>
       <axis xyz="0 0 1"/>
-      <limit lower="-2.0" upper="0.0" velocity="2.0" effort="1000" />
+      <limit lower="-2.3" upper="-0.05" velocity="2.0" effort="1000" />
     </joint>
   </xacro:macro>

File: avatar_robot_description/franka/common/franka_arm.xacro (robot description, xacro)
@@ -1,9 +1,9 @@
 <?xml version='1.0' encoding='utf-8'?>
 <robot xmlns:xacro="http://www.ros.org/wiki/xacro" name="panda">
-  <xacro:include filename="$(find franka_description)/robots/common/utils.xacro" />
+  <xacro:include filename="$(find avatar_robot_description)/franka/common/utils.xacro" />
   <!-- safety_distance: Minimum safety distance in [m] by which the collision volumes are expanded and which is enforced during robot motions -->
   <!-- arm_id: Namespace of the robot arm. Serves to differentiate between arms in case of multiple instances. -->
   <!-- joint_limits: description of the joint limits that comes from a YAML file. Example definition: ${xacro.load_yaml('$(find franka_description)/robots/fr3/joint_limits.yaml')} -->
-  <xacro:macro name="franka_arm" params="arm_id:='panda' description_pkg:='franka_description' connected_to:='' xyz:='0 0 0' rpy:='0 0 0' gazebo:=false safety_distance:=0 joint_limits" >
+  <xacro:macro name="franka_arm" params="arm_id:='panda' description_pkg:='avatar_robot_description' connected_to:='' xyz:='0 0 0' rpy:='0 0 0' gazebo:=false safety_distance:=0 joint_limits" >
     <xacro:unless value="${not connected_to}">
       <joint name="${arm_id}_joint_${connected_to}" type="fixed">

File: avatar_robot_description/franka/common/franka_robot.xacro (robot description, xacro)
@@ -11,6 +11,6 @@
     <!-- Is the robot being simulated in gazebo?" -->
     <xacro:arg name="gazebo" default="false" />
-    <xacro:include filename="$(find franka_description)/robots/common/utils.xacro" />
-    <xacro:include filename="$(find franka_description)/robots/common/franka_arm.xacro" />
+    <xacro:include filename="$(find avatar_robot_description)/franka/common/utils.xacro" />
+    <xacro:include filename="$(find avatar_robot_description)/franka/common/franka_arm.xacro" />
     <xacro:franka_arm arm_id="${arm_id}" safety_distance="0.03" gazebo="$(arg gazebo)" joint_limits="${joint_limits}"/>
     <xacro:if value="$(arg hand)">

File: avatar_robot_description/franka/common/utils.xacro (robot description, xacro)
@@ -2,5 +2,5 @@
 <robot xmlns:xacro="http://www.ros.org/wiki/xacro">
   <!-- Load inertial properties. Property is implicitly passed to macros. -->
-  <xacro:property name="inertial_config" value="$(find franka_description)/robots/common/inertial.yaml"/>
+  <xacro:property name="inertial_config" value="$(find avatar_robot_description)/franka/common/inertial.yaml"/>
   <xacro:property name="inertial" value="${xacro.load_yaml(inertial_config)}"/>
   <!-- ============================================================== -->
@@ -43,5 +43,5 @@
       <collision>
         <geometry>
-          <mesh filename="package://franka_description/meshes/collision/${name}.stl" />
+          <mesh filename="package://avatar_robot_description/meshes/collision/${name}.stl" />
         </geometry>
       </collision>

Commit message: linearization model value change

File: avatar_gripper_description/urdf/avatar_gripper_3f_macro.xacro (robot description, xacro)
@@ -260,5 +260,5 @@
       <axis xyz="0 0 1"/>
       <limit lower="-0.8" upper="0" velocity="2.0" effort="1000" />
-      <mimic joint="${prefix}_index_flex_motor_joint" offsite="0" multiplier="0.6"/>
+      <mimic joint="${prefix}_index_flex_motor_joint" offsite="0" multiplier="0.4"/>
     </joint>
   </xacro:macro>

Commit message: typo fix

File: avatar_gripper_description/urdf/avatar_gripper_3f_macro.xacro (robot description, xacro)
@@ -213,5 +213,5 @@
       <axis xyz="0 1 0"/>
       <limit lower="-1.0" upper="0.4" velocity="2.0" effort="1000" />
-      <mimic joint="${prefix}_thumb_flex_motor_joint" offsite="0" multiplier="0.28"/>
+      <mimic joint="${prefix}_thumb_flex_motor_joint" offset="0" multiplier="0.28"/>
     </joint>
   </xacro:macro>
@@ -223,5 +223,5 @@
       <axis xyz="0 1 0"/>
       <limit lower="-0.8" upper="0" velocity="2.0" effort="1000" />
-      <mimic joint="${prefix}_thumb_flex_motor_joint" offsite="0" multiplier="0.24"/>
+      <mimic joint="${prefix}_thumb_flex_motor_joint" offset="0" multiplier="0.24"/>
     </joint>
   </xacro:macro>
@@ -250,5 +250,5 @@
       <axis xyz="0 0 1"/>
       <limit lower="-0.8" upper="0" velocity="2.0" effort="1000" />
-      <mimic joint="${prefix}_index_flex_motor_joint" offsite="0" multiplier="0.4016"/>
+      <mimic joint="${prefix}_index_flex_motor_joint" offset="0" multiplier="0.4016"/>
     </joint>
   </xacro:macro>
@@ -260,5 +260,5 @@
       <axis xyz="0 0 1"/>
       <limit lower="-0.8" upper="0" velocity="2.0" effort="1000" />
-      <mimic joint="${prefix}_index_flex_motor_joint" offsite="0" multiplier="0.4"/>
+      <mimic joint="${prefix}_index_flex_motor_joint" offset="0" multiplier="0.4"/>
     </joint>
   </xacro:macro>

Commit message: used STL instead of OBJ for Unity support

File: avatar_gripper_description/urdf/avatar_gripper_3f_macro.xacro (robot description, xacro)
@@ -10,5 +10,5 @@
         <origin xyz="0 0 0" rpy="0 0 0"/>
         <geometry>
-          <mesh filename="package://avatar_gripper_description/meshes/${prefix}/gripper_base.obj"/>
+          <mesh filename="package://avatar_gripper_description/meshes/${prefix}/gripper_base.STL"/>
         </geometry>
         <material name="">
@@ -16,4 +16,10 @@
         </material>
       </visual>
+      <collision>
+        <origin xyz="0 0 -0.03" rpy="0 0 0"/>
+        <geometry>
+          <box size="0.1 0.1 0.06"/>
+        </geometry>
+      </collision>
     </link>
   </xacro:macro>
@@ -22,19 +28,19 @@
       <inertial>
         <mass value="0.5"/>
-        <inertia ixx="0.0" ixy="0.0" ixz="0.0" iyy="4E-5" iyz="0.0" izz="4E-5"/>
-      </inertial>
-      <visual>
-        <origin xyz="0 0 0" rpy="0 0 0"/>
-        <geometry>
-          <mesh filename="package://avatar_gripper_description/meshes/${prefix}/thumb_base_extra.obj"/>
-        </geometry>
-        <material name="">
-          <color rgba="0.9 0.9 0.9 1"/>
-        </material>
-      </visual>
-      <collision>
-        <origin xyz="0 0 0" rpy="0 0 0"/>
-        <geometry>
-          <mesh filename="package://avatar_gripper_description/meshes/${prefix}/thumb_base_extra.obj"/>
+        <inertia ixx="4E-5" ixy="0.0" ixz="0.0" iyy="4E-5" iyz="0.0" izz="4E-5"/>
+      </inertial>
+      <visual>
+        <origin xyz="0 0 0" rpy="0 0 0"/>
+        <geometry>
+          <mesh filename="package://avatar_gripper_description/meshes/${prefix}/thumb_base_extra.STL"/>
+        </geometry>
+        <material name="">
+          <color rgba="0.9 0.9 0.9 1"/>
+        </material>
+      </visual>
+      <collision>
+        <origin xyz="0 0 0" rpy="0 0 0"/>
+        <geometry>
+          <mesh filename="package://avatar_gripper_description/meshes/${prefix}/thumb_base_extra.STL"/>
         </geometry>
       </collision>
@@ -45,19 +51,19 @@
       <inertial>
         <mass value="0.5"/>
-        <inertia ixx="0.0" ixy="0.0" ixz="0.0" iyy="4E-5" iyz="0.0" izz="4E-5"/>
-      </inertial>
-      <visual>
-        <origin xyz="0 0 0" rpy="0 0 0"/>
-        <geometry>
-          <mesh filename="package://avatar_gripper_description/meshes/${prefix}/thumb_knuckle.obj"/>
-        </geometry>
-        <material name="">
-          <color rgba="0.9 0.9 0.9 1"/>
-        </material>
-      </visual>
-      <collision>
-        <origin xyz="0 0 0" rpy="0 0 0"/>
-        <geometry>
-          <mesh filename="package://avatar_gripper_description/meshes/${prefix}/thumb_knuckle.obj"/>
+        <inertia ixx="4E-5" ixy="0.0" ixz="0.0" iyy="4E-5" iyz="0.0" izz="4E-5"/>
+      </inertial>
+      <visual>
+        <origin xyz="0 0 0" rpy="0 0 0"/>
+        <geometry>
+          <mesh filename="package://avatar_gripper_description/meshes/${prefix}/thumb_knuckle.STL"/>
+        </geometry>
+        <material name="">
+          <color rgba="0.9 0.9 0.9 1"/>
+        </material>
+      </visual>
+      <collision>
+        <origin xyz="0 0 0" rpy="0 0 0"/>
+        <geometry>
+          <mesh filename="package://avatar_gripper_description/meshes/${prefix}/thumb_knuckle.STL"/>
         </geometry>
       </collision>
@@ -68,19 +74,19 @@
       <inertial>
         <mass value="0.5"/>
-        <inertia ixx="0.0" ixy="0.0" ixz="0.0" iyy="4E-5" iyz="0.0" izz="4E-5"/>
-      </inertial>
-      <visual>
-        <origin xyz="0 0 0" rpy="0 0 0"/>
-        <geometry>
-          <mesh filename="package://avatar_gripper_description/meshes/${prefix}/thumb_fingertip.obj"/>
-        </geometry>
-        <material name="">
-          <color rgba="0.9 0.9 0.9 1"/>
-        </material>
-      </visual>
-      <collision>
-        <origin xyz="0 0 0" rpy="0 0 0"/>
-        <geometry>
-          <mesh filename="package://avatar_gripper_description/meshes/${prefix}/thumb_fingertip.obj"/>
+        <inertia ixx="4E-5" ixy="0.0" ixz="0.0" iyy="4E-5" iyz="0.0" izz="4E-5"/>
+      </inertial>
+      <visual>
+        <origin xyz="0 0 0" rpy="0 0 0"/>
+        <geometry>
+          <mesh filename="package://avatar_gripper_description/meshes/${prefix}/thumb_fingertip.STL"/>
+        </geometry>
+        <material name="">
+          <color rgba="0.9 0.9 0.9 1"/>
+        </material>
+      </visual>
+      <collision>
+        <origin xyz="0 0 0" rpy="0 0 0"/>
+        <geometry>
+          <mesh filename="package://avatar_gripper_description/meshes/${prefix}/thumb_fingertip.STL"/>
         </geometry>
       </collision>
@@ -89,8 +95,12 @@
   <xacro:macro name="index_base_connector" params="prefix">
     <link name="${prefix}_index_base_connector">
-      <visual>
-        <origin xyz="0 0 0" rpy="0 0 0"/>
-        <geometry>
-          <mesh filename="package://avatar_gripper_description/meshes/${prefix}/index_base_connector.obj"/>
+      <inertial>
+        <mass value="0.02"/>
+        <inertia ixx="4E-5" ixy="0.0" ixz="0.0" iyy="4E-5" iyz="0.0" izz="4E-5"/>
+      </inertial>
+      <visual>
+        <origin xyz="0 0 0" rpy="0 0 0"/>
+        <geometry>
+          <mesh filename="package://avatar_gripper_description/meshes/${prefix}/index_base_connector.STL"/>
         </geometry>
         <material name="">
@@ -104,19 +114,19 @@
       <inertial>
         <mass value="0.5"/>
-        <inertia ixx="0.0" ixy="0.0" ixz="0.0" iyy="4E-5" iyz="0.0" izz="4E-5"/>
-      </inertial>
-      <visual>
-        <origin xyz="0 0 0" rpy="0 0 0"/>
-        <geometry>
-          <mesh filename="package://avatar_gripper_description/meshes/${prefix}/index_knuckle.obj"/>
-        </geometry>
-        <material name="">
-          <color rgba="0.9 0.9 0.9 1"/>
-        </material>
-      </visual>
-      <collision>
-        <origin xyz="0 0 0" rpy="0 0 0"/>
-        <geometry>
-          <mesh filename="package://avatar_gripper_description/meshes/${prefix}/index_knuckle.obj"/>
+        <inertia ixx="4E-5" ixy="0.0" ixz="0.0" iyy="4E-5" iyz="0.0" izz="4E-5"/>
+      </inertial>
+      <visual>
+        <origin xyz="0 0 0" rpy="0 0 0"/>
+        <geometry>
+          <mesh filename="package://avatar_gripper_description/meshes/${prefix}/index_knuckle.STL"/>
+        </geometry>
+        <material name="">
+          <color rgba="0.9 0.9 0.9 1"/>
+        </material>
+      </visual>
+      <collision>
+        <origin xyz="0 0 0" rpy="0 0 0"/>
+        <geometry>
+          <mesh filename="package://avatar_gripper_description/meshes/${prefix}/index_knuckle.STL"/>
         </geometry>
       </collision>
@@ -127,19 +137,19 @@
       <inertial>
         <mass value="0.5"/>
-        <inertia ixx="0.0" ixy="0.0" ixz="0.0" iyy="4E-5" iyz="0.0" izz="4E-5"/>
-      </inertial>
-      <visual>
-        <origin xyz="0 0 0" rpy="0 0 0"/>
-        <geometry>
-          <mesh filename="package://avatar_gripper_description/meshes/${prefix}/index_fingertip.obj"/>
-        </geometry>
-        <material name="">
-          <color rgba="0.9 0.9 0.9 1"/>
-        </material>
-      </visual>
-      <collision>
-        <origin xyz="0 0 0" rpy="0 0 0"/>
-        <geometry>
-          <mesh filename="package://avatar_gripper_description/meshes/${prefix}/index_fingertip.obj"/>
+        <inertia ixx="4E-5" ixy="0.0" ixz="0.0" iyy="4E-5" iyz="0.0" izz="4E-5"/>
+      </inertial>
+      <visual>
+        <origin xyz="0 0 0" rpy="0 0 0"/>
+        <geometry>
+          <mesh filename="package://avatar_gripper_description/meshes/${prefix}/index_fingertip.STL"/>
+        </geometry>
+        <material name="">
+          <color rgba="0.9 0.9 0.9 1"/>
+        </material>
+      </visual>
+      <collision>
+        <origin xyz="0 0 0" rpy="0 0 0"/>
+        <geometry>
+          <mesh filename="package://avatar_gripper_description/meshes/${prefix}/index_fingertip.STL"/>
         </geometry>
       </collision>
@@ -150,19 +160,19 @@
       <inertial>
         <mass value="0.5"/>
-        <inertia ixx="0.0" ixy="0.0" ixz="0.0" iyy="4E-5" iyz="0.0" izz="4E-5"/>
-      </inertial>
-      <visual>
-        <origin xyz="0 0 0" rpy="0 0 0"/>
-        <geometry>
-          <mesh filename="package://avatar_gripper_description/meshes/${prefix}/index_knuckle.obj"/>
-        </geometry>
-        <material name="">
-          <color rgba="0.9 0.9 0.9 1"/>
-        </material>
-      </visual>
-      <collision>
-        <origin xyz="0 0 0" rpy="0 0 0"/>
-        <geometry>
-          <mesh filename="package://avatar_gripper_description/meshes/${prefix}/index_knuckle.obj"/>
+        <inertia ixx="4E-5" ixy="0.0" ixz="0.0" iyy="4E-5" iyz="0.0" izz="4E-5"/>
+      </inertial>
+      <visual>
+        <origin xyz="0 0 0" rpy="0 0 0"/>
+        <geometry>
+          <mesh filename="package://avatar_gripper_description/meshes/${prefix}/index_knuckle.STL"/>
+        </geometry>
+        <material name="">
+          <color rgba="0.9 0.9 0.9 1"/>
+        </material>
+      </visual>
+      <collision>
+        <origin xyz="0 0 0" rpy="0 0 0"/>
+        <geometry>
+          <mesh filename="package://avatar_gripper_description/meshes/${prefix}/index_knuckle.STL"/>
         </geometry>
       </collision>
@@ -173,19 +183,19 @@
       <inertial>
         <mass value="0.5"/>
-        <inertia ixx="0.0" ixy="0.0" ixz="0.0" iyy="4E-5" iyz="0.0" izz="4E-5"/>
-      </inertial>
-      <visual>
-        <origin xyz="0 0 0" rpy="0 0 0"/>
-        <geometry>
-          <mesh filename="package://avatar_gripper_description/meshes/${prefix}/index_fingertip.obj"/>
-        </geometry>
-        <material name="">
-          <color rgba="0.9 0.9 0.9 1"/>
-        </material>
-      </visual>
-      <collision>
-        <origin xyz="0 0 0" rpy="0 0 0"/>
-        <geometry>
-          <mesh filename="package://avatar_gripper_description/meshes/${prefix}/index_fingertip.obj"/>
+        <inertia ixx="4E-5" ixy="0.0" ixz="0.0" iyy="4E-5" iyz="0.0" izz="4E-5"/>
+      </inertial>
+      <visual>
+        <origin xyz="0 0 0" rpy="0 0 0"/>
+        <geometry>
+          <mesh filename="package://avatar_gripper_description/meshes/${prefix}/index_fingertip.STL"/>
+        </geometry>
+        <material name="">
+          <color rgba="0.9 0.9 0.9 1"/>
+        </material>
+      </visual>
+      <collision>
+        <origin xyz="0 0 0" rpy="0 0 0"/>
+        <geometry>
+          <mesh filename="package://avatar_gripper_description/meshes/${prefix}/index_fingertip.STL"/>
         </geometry>
       </collision>
@@ -194,13 +204,23 @@
   <xacro:macro name="thumb_swivel_link" params="prefix">
     <link name="${prefix}_thumb_swivel_link">
-      <visual>
-        <origin xyz="0 0 0" rpy="0 0 0"/>
-        <geometry>
-          <mesh filename="package://avatar_gripper_description/meshes/${prefix}/thumb_swivel_link.obj"/>
-        </geometry>
-        <material name="">
-          <color rgba="0.9 0.9 0.9 1"/>
-        </material>
-      </visual>
+      <inertial>
+        <mass value="0.1"/>
+        <inertia ixx="4E-5" ixy="0.0" ixz="0.0" iyy="4E-5" iyz="0.0" izz="4E-5"/>
+      </inertial>
+      <visual>
+        <origin xyz="0 0 0" rpy="0 0 0"/>
+        <geometry>
+          <mesh filename="package://avatar_gripper_description/meshes/${prefix}/thumb_swivel_link.STL"/>
+        </geometry>
+        <material name="">
+          <color rgba="0.9 0.9 0.9 1"/>
+        </material>
+      </visual>
+      <collision>
+        <origin xyz="0 0 0" rpy="0 0 0"/>
+        <geometry>
+          <mesh filename="package://avatar_gripper_description/meshes/${prefix}/thumb_swivel_link.STL"/>
+        </geometry>
+      </collision>
     </link>
   </xacro:macro>
