Commit message: used STL instead of OBJ for Unity support

File: avatar_gripper_description/urdf/avatar_gripper_3f_macro_nomimic.xacro (robot description, xacro)
@@ -10,5 +10,5 @@
         <origin xyz="0 0 0" rpy="0 0 0"/>
         <geometry>
-          <mesh filename="package://avatar_gripper_description/meshes/${prefix}/gripper_base.obj"/>
+          <mesh filename="package://avatar_gripper_description/meshes/${prefix}/gripper_base.STL"/>
         </geometry>
         <material name="">
@@ -16,4 +16,10 @@
         </material>
       </visual>
+      <collision>
+        <origin xyz="0 0 -0.03" rpy="0 0 0"/>
+        <geometry>
+          <box size="0.1 0.1 0.06"/>
+        </geometry>
+      </collision>
     </link>
   </xacro:macro>
@@ -22,19 +28,19 @@
       <inertial>
         <mass value="0.5"/>
-        <inertia ixx="0.0" ixy="0.0" ixz="0.0" iyy="4E-5" iyz="0.0" izz="4E-5"/>
-      </inertial>
-      <visual>
-        <origin xyz="0 0 0" rpy="0 0 0"/>
-        <geometry>
-          <mesh filename="package://avatar_gripper_description/meshes/${prefix}/thumb_base_extra.obj"/>
-        </geometry>
-        <material name="">
-          <color rgba="0.9 0.9 0.9 1"/>
-        </material>
-      </visual>
-      <collision>
-        <origin xyz="0 0 0" rpy="0 0 0"/>
-        <geometry>
-          <mesh filename="package://avatar_gripper_description/meshes/${prefix}/thumb_base_extra.obj"/>
+        <inertia ixx="4E-5" ixy="0.0" ixz="0.0" iyy="4E-5" iyz="0.0" izz="4E-5"/>
+      </inertial>
+      <visual>
+        <origin xyz="0 0 0" rpy="0 0 0"/>
+        <geometry>
+          <mesh filename="package://avatar_gripper_description/meshes/${prefix}/thumb_base_extra.STL"/>
+        </geometry>
+        <material name="">
+          <color rgba="0.9 0.9 0.9 1"/>
+        </material>
+      </visual>
+      <collision>
+        <origin xyz="0 0 0" rpy="0 0 0"/>
+        <geometry>
+          <mesh filename="package://avatar_gripper_description/meshes/${prefix}/thumb_base_extra.STL"/>
         </geometry>
       </collision>
@@ -45,19 +51,19 @@
       <inertial>
         <mass value="0.5"/>
-        <inertia ixx="0.0" ixy="0.0" ixz="0.0" iyy="4E-5" iyz="0.0" izz="4E-5"/>
-      </inertial>
-      <visual>
-        <origin xyz="0 0 0" rpy="0 0 0"/>
-        <geometry>
-          <mesh filename="package://avatar_gripper_description/meshes/${prefix}/thumb_knuckle.obj"/>
-        </geometry>
-        <material name="">
-          <color rgba="0.9 0.9 0.9 1"/>
-        </material>
-      </visual>
-      <collision>
-        <origin xyz="0 0 0" rpy="0 0 0"/>
-        <geometry>
-          <mesh filename="package://avatar_gripper_description/meshes/${prefix}/thumb_knuckle.obj"/>
+        <inertia ixx="4E-5" ixy="0.0" ixz="0.0" iyy="4E-5" iyz="0.0" izz="4E-5"/>
+      </inertial>
+      <visual>
+        <origin xyz="0 0 0" rpy="0 0 0"/>
+        <geometry>
+          <mesh filename="package://avatar_gripper_description/meshes/${prefix}/thumb_knuckle.STL"/>
+        </geometry>
+        <material name="">
+          <color rgba="0.9 0.9 0.9 1"/>
+        </material>
+      </visual>
+      <collision>
+        <origin xyz="0 0 0" rpy="0 0 0"/>
+        <geometry>
+          <mesh filename="package://avatar_gripper_description/meshes/${prefix}/thumb_knuckle.STL"/>
         </geometry>
       </collision>
@@ -68,19 +74,19 @@
       <inertial>
         <mass value="0.5"/>
-        <inertia ixx="0.0" ixy="0.0" ixz="0.0" iyy="4E-5" iyz="0.0" izz="4E-5"/>
-      </inertial>
-      <visual>
-        <origin xyz="0 0 0" rpy="0 0 0"/>
-        <geometry>
-          <mesh filename="package://avatar_gripper_description/meshes/${prefix}/thumb_fingertip.obj"/>
-        </geometry>
-        <material name="">
-          <color rgba="0.9 0.9 0.9 1"/>
-        </material>
-      </visual>
-      <collision>
-        <origin xyz="0 0 0" rpy="0 0 0"/>
-        <geometry>
-          <mesh filename="package://avatar_gripper_description/meshes/${prefix}/thumb_fingertip.obj"/>
+        <inertia ixx="4E-5" ixy="0.0" ixz="0.0" iyy="4E-5" iyz="0.0" izz="4E-5"/>
+      </inertial>
+      <visual>
+        <origin xyz="0 0 0" rpy="0 0 0"/>
+        <geometry>
+          <mesh filename="package://avatar_gripper_description/meshes/${prefix}/thumb_fingertip.STL"/>
+        </geometry>
+        <material name="">
+          <color rgba="0.9 0.9 0.9 1"/>
+        </material>
+      </visual>
+      <collision>
+        <origin xyz="0 0 0" rpy="0 0 0"/>
+        <geometry>
+          <mesh filename="package://avatar_gripper_description/meshes/${prefix}/thumb_fingertip.STL"/>
         </geometry>
       </collision>
@@ -89,8 +95,12 @@
   <xacro:macro name="index_base_connector" params="prefix">
     <link name="${prefix}_index_base_connector">
-      <visual>
-        <origin xyz="0 0 0" rpy="0 0 0"/>
-        <geometry>
-          <mesh filename="package://avatar_gripper_description/meshes/${prefix}/index_base_connector.obj"/>
+      <inertial>
+        <mass value="0.02"/>
+        <inertia ixx="4E-5" ixy="0.0" ixz="0.0" iyy="4E-5" iyz="0.0" izz="4E-5"/>
+      </inertial>
+      <visual>
+        <origin xyz="0 0 0" rpy="0 0 0"/>
+        <geometry>
+          <mesh filename="package://avatar_gripper_description/meshes/${prefix}/index_base_connector.STL"/>
         </geometry>
         <material name="">
@@ -104,19 +114,19 @@
       <inertial>
         <mass value="0.5"/>
-        <inertia ixx="0.0" ixy="0.0" ixz="0.0" iyy="4E-5" iyz="0.0" izz="4E-5"/>
-      </inertial>
-      <visual>
-        <origin xyz="0 0 0" rpy="0 0 0"/>
-        <geometry>
-          <mesh filename="package://avatar_gripper_description/meshes/${prefix}/index_knuckle.obj"/>
-        </geometry>
-        <material name="">
-          <color rgba="0.9 0.9 0.9 1"/>
-        </material>
-      </visual>
-      <collision>
-        <origin xyz="0 0 0" rpy="0 0 0"/>
-        <geometry>
-          <mesh filename="package://avatar_gripper_description/meshes/${prefix}/index_knuckle.obj"/>
+        <inertia ixx="4E-5" ixy="0.0" ixz="0.0" iyy="4E-5" iyz="0.0" izz="4E-5"/>
+      </inertial>
+      <visual>
+        <origin xyz="0 0 0" rpy="0 0 0"/>
+        <geometry>
+          <mesh filename="package://avatar_gripper_description/meshes/${prefix}/index_knuckle.STL"/>
+        </geometry>
+        <material name="">
+          <color rgba="0.9 0.9 0.9 1"/>
+        </material>
+      </visual>
+      <collision>
+        <origin xyz="0 0 0" rpy="0 0 0"/>
+        <geometry>
+          <mesh filename="package://avatar_gripper_description/meshes/${prefix}/index_knuckle.STL"/>
         </geometry>
       </collision>
@@ -127,19 +137,19 @@
       <inertial>
         <mass value="0.5"/>
-        <inertia ixx="0.0" ixy="0.0" ixz="0.0" iyy="4E-5" iyz="0.0" izz="4E-5"/>
-      </inertial>
-      <visual>
-        <origin xyz="0 0 0" rpy="0 0 0"/>
-        <geometry>
-          <mesh filename="package://avatar_gripper_description/meshes/${prefix}/index_fingertip.obj"/>
-        </geometry>
-        <material name="">
-          <color rgba="0.9 0.9 0.9 1"/>
-        </material>
-      </visual>
-      <collision>
-        <origin xyz="0 0 0" rpy="0 0 0"/>
-        <geometry>
-          <mesh filename="package://avatar_gripper_description/meshes/${prefix}/index_fingertip.obj"/>
+        <inertia ixx="4E-5" ixy="0.0" ixz="0.0" iyy="4E-5" iyz="0.0" izz="4E-5"/>
+      </inertial>
+      <visual>
+        <origin xyz="0 0 0" rpy="0 0 0"/>
+        <geometry>
+          <mesh filename="package://avatar_gripper_description/meshes/${prefix}/index_fingertip.STL"/>
+        </geometry>
+        <material name="">
+          <color rgba="0.9 0.9 0.9 1"/>
+        </material>
+      </visual>
+      <collision>
+        <origin xyz="0 0 0" rpy="0 0 0"/>
+        <geometry>
+          <mesh filename="package://avatar_gripper_description/meshes/${prefix}/index_fingertip.STL"/>
         </geometry>
       </collision>
@@ -150,19 +160,19 @@
       <inertial>
         <mass value="0.5"/>
-        <inertia ixx="0.0" ixy="0.0" ixz="0.0" iyy="4E-5" iyz="0.0" izz="4E-5"/>
-      </inertial>
-      <visual>
-        <origin xyz="0 0 0" rpy="0 0 0"/>
-        <geometry>
-          <mesh filename="package://avatar_gripper_description/meshes/${prefix}/index_knuckle.obj"/>
-        </geometry>
-        <material name="">
-          <color rgba="0.9 0.9 0.9 1"/>
-        </material>
-      </visual>
-      <collision>
-        <origin xyz="0 0 0" rpy="0 0 0"/>
-        <geometry>
-          <mesh filename="package://avatar_gripper_description/meshes/${prefix}/index_knuckle.obj"/>
+        <inertia ixx="4E-5" ixy="0.0" ixz="0.0" iyy="4E-5" iyz="0.0" izz="4E-5"/>
+      </inertial>
+      <visual>
+        <origin xyz="0 0 0" rpy="0 0 0"/>
+        <geometry>
+          <mesh filename="package://avatar_gripper_description/meshes/${prefix}/index_knuckle.STL"/>
+        </geometry>
+        <material name="">
+          <color rgba="0.9 0.9 0.9 1"/>
+        </material>
+      </visual>
+      <collision>
+        <origin xyz="0 0 0" rpy="0 0 0"/>
+        <geometry>
+          <mesh filename="package://avatar_gripper_description/meshes/${prefix}/index_knuckle.STL"/>
         </geometry>
       </collision>
@@ -173,20 +183,20 @@
       <inertial>
         <mass value="0.5"/>
-        <inertia ixx="0.0" ixy="0.0" ixz="0.0" iyy="4E-5" iyz="0.0" izz="4E-5"/>
-      </inertial>
-      <visual>
-        <origin xyz="0 0 0" rpy="0 0 0"/>
-        <geometry>
-          <mesh filename="package://avatar_gripper_description/meshes/${prefix}/index_fingertip.obj"/>
-        </geometry>
-        <material name="">
-          <color rgba="0.9 0.9 0.9 1"/>
-        </material>
-      </visual>
-      <collision>
-        <geometry>
-          <mesh filename="package://avatar_gripper_description/meshes/${prefix}/index_fingertip.obj"/>
-        </geometry>
-        <origin xyz="0 0 0" rpy="0 0 0"/>
+        <inertia ixx="4E-5" ixy="0.0" ixz="0.0" iyy="4E-5" iyz="0.0" izz="4E-5"/>
+      </inertial>
+      <visual>
+        <origin xyz="0 0 0" rpy="0 0 0"/>
+        <geometry>
+          <mesh filename="package://avatar_gripper_description/meshes/${prefix}/index_fingertip.STL"/>
+        </geometry>
+        <material name="">
+          <color rgba="0.9 0.9 0.9 1"/>
+        </material>
+      </visual>
+      <collision>
+        <origin xyz="0 0 0" rpy="0 0 0"/>
+        <geometry>
+          <mesh filename="package://avatar_gripper_description/meshes/${prefix}/index_fingertip.STL"/>
+        </geometry>
       </collision>
     </link>
@@ -194,13 +204,23 @@
   <xacro:macro name="thumb_swivel_link" params="prefix">
     <link name="${prefix}_thumb_swivel_link">
-      <visual>
-        <origin xyz="0 0 0" rpy="0 0 0"/>
-        <geometry>
-          <mesh filename="package://avatar_gripper_description/meshes/${prefix}/thumb_swivel_link.obj"/>
-        </geometry>
-        <material name="">
-          <color rgba="0.9 0.9 0.9 1"/>
-        </material>
-      </visual>
+      <inertial>
+        <mass value="0.1"/>
+        <inertia ixx="4E-5" ixy="0.0" ixz="0.0" iyy="4E-5" iyz="0.0" izz="4E-5"/>
+      </inertial>
+      <visual>
+        <origin xyz="0 0 0" rpy="0 0 0"/>
+        <geometry>
+          <mesh filename="package://avatar_gripper_description/meshes/${prefix}/thumb_swivel_link.STL"/>
+        </geometry>
+        <material name="">
+          <color rgba="0.9 0.9 0.9 1"/>
+        </material>
+      </visual>
+      <collision>
+        <origin xyz="0 0 0" rpy="0 0 0"/>
+        <geometry>
+          <mesh filename="package://avatar_gripper_description/meshes/${prefix}/thumb_swivel_link.STL"/>
+        </geometry>
+      </collision>
     </link>
   </xacro:macro>

File: avatar_robot_description/franka/dual_panda/dual_panda_example.urdf.xacro (robot description, xacro)
@@ -1,17 +1,18 @@
 <?xml version="1.0" encoding="utf-8"?>
-<robot xmlns:xacro="http://www.ros.org/wiki/xacro" name="panda">
+<robot xmlns:xacro="http://www.ros.org/wiki/xacro" name="avatar">
   <xacro:arg name="arm_id_1" default="right_panda" />
   <xacro:arg name="arm_id_2" default="left_panda" />
   <xacro:arg name="pref_1" default="right" />
   <xacro:arg name="pref_2" default="left" />
+  <xacro:arg name="gazebo" default="true"/>
   <xacro:include filename="$(find avatar_robot_description)/franka/common/franka_arm.xacro"/>
   <xacro:include filename="$(find avatar_robot_description)/franka/common/base.xacro"/>
   <xacro:include filename="$(find avatar_gripper_description)/urdf/avatar_gripper_3f.xacro"/>
   <!-- right arm with gripper -->
-  <xacro:franka_arm arm_id="$(arg arm_id_1)" connected_to="support"  xyz="${length_support*0.45} ${-dist_arms/2} ${heigth_support/2}" rpy='0 0 0' safety_distance="0.03" joint_limits="${xacro.load_yaml('$(find avatar_robot_description)/franka/panda/joint_limits.yaml')}"/>
+  <xacro:franka_arm arm_id="$(arg arm_id_1)" connected_to="support" gazebo="$(arg gazebo)" xyz="${length_support*0.45} ${-dist_arms/2} ${heigth_support/2}" rpy='0 0 0' safety_distance="0.03" joint_limits="${xacro.load_yaml('$(find avatar_robot_description)/franka/panda/joint_limits.yaml')}"/>
   <xacro:avatar_gripper_3f prefix="$(arg pref_1)"/>
   <xacro:attach_gripper connected_to="$(arg arm_id_1)_link8" arm_id="$(arg arm_id_1)" gripper_prefix='right' rpy="0 ${pi} ${-pi/4}" xyz='0 0 0'/>
   <!-- left arm with gripper -->
-  <xacro:franka_arm arm_id="$(arg arm_id_2)" connected_to="support"  xyz="${length_support*0.45} ${dist_arms/2} ${heigth_support/2}" rpy='0 0 0' safety_distance="0.03" joint_limits="${xacro.load_yaml('$(find avatar_robot_description)/franka/panda/joint_limits.yaml')}"/>
+  <xacro:franka_arm arm_id="$(arg arm_id_2)" connected_to="support"  gazebo="$(arg gazebo)" xyz="${length_support*0.45} ${dist_arms/2} ${heigth_support/2}" rpy='0 0 0' safety_distance="0.03" joint_limits="${xacro.load_yaml('$(find avatar_robot_description)/franka/panda/joint_limits.yaml')}"/>
   <xacro:avatar_gripper_3f prefix="$(arg pref_2)"/>
   <xacro:attach_gripper connected_to="$(arg arm_id_2)_link8" arm_id="$(arg arm_id_2)" gripper_prefix='left' rpy="0 ${pi} ${-pi/4}" xyz='0 0 0'/>

Commit message: Corrected thumb knuckle STL file.

File: avatar_gripper_description/urdf/avatar_gripper_3f_macro.xacro (robot description, xacro)
@@ -108,4 +108,13 @@
         </material>
       </visual>
+      <collision>
+        <origin xyz="0 0 0" rpy="0 0 0"/>
+        <geometry>
+          <mesh filename="package://avatar_gripper_description/meshes/${prefix}/index_base_connector.STL"/>
+        </geometry>
+        <material name="">
+          <color rgba="0.9 0.9 0.9 1"/>
+        </material>
+      </collision>
     </link>
   </xacro:macro>
