Commit message: replaced all mesh collision file for gripper with capsule collision primitive

File: avatar_gripper_description/urdf/avatar_gripper_3f_macro.xacro (robot description, xacro)
@@ -1,4 +1,5 @@
 <?xml version="1.0"?>
 <robot xmlns:xacro="http://ros.org/wiki/xacro">
+  <xacro:include filename="$(find avatar_gripper_description)/urdf/utils.xacro"/>
   <xacro:macro name="gripper_base_link" params="prefix">
     <link name="${prefix}_gripper_base">
@@ -10,5 +11,5 @@
         <origin xyz="0 0 0" rpy="0 0 0"/>
         <geometry>
-          <mesh filename="package://avatar_gripper_description/meshes/${prefix}/gripper_base.STL"/>
+          <mesh filename="package://avatar_gripper_description/meshes/${prefix}/gripper_base.obj"/>
         </geometry>
         <material name="">
@@ -16,10 +17,10 @@
         </material>
       </visual>
-      <collision>
+      <!-- <collision>
         <origin xyz="0 0 -0.03" rpy="0 0 0"/>
         <geometry>
           <box size="0.1 0.1 0.06"/>
         </geometry>
-      </collision>
+      </collision> -->
     </link>
   </xacro:macro>
@@ -31,18 +32,13 @@
       </inertial>
       <visual>
-        <origin xyz="0 0 0" rpy="0 0 0"/>
-        <geometry>
-          <mesh filename="package://avatar_gripper_description/meshes/${prefix}/thumb_base_extra.STL"/>
-        </geometry>
-        <material name="">
-          <color rgba="0.9 0.9 0.9 1"/>
-        </material>
-      </visual>
-      <collision>
-        <origin xyz="0 0 0" rpy="0 0 0"/>
-        <geometry>
-          <mesh filename="package://avatar_gripper_description/meshes/${prefix}/thumb_base_extra.STL"/>
-        </geometry>
-      </collision>
+        <origin xyz="0 0 0" rpy="0 0   0"/>
+        <geometry>
+          <mesh filename="package://avatar_gripper_description/meshes/${prefix}/thumb_base_extra.obj"/>
+        </geometry>
+        <material name="">
+          <color rgba="0.9 0.9 0.9 1"/>
+        </material>
+      </visual>
+      <xacro:collision_capsule_custom radius="0.01" length="0.036" xyz="0 0 -0.02" direction="z 0"/>
     </link>
   </xacro:macro>
@@ -56,16 +52,17 @@
         <origin xyz="0 0 0" rpy="0 0 0"/>
         <geometry>
-          <mesh filename="package://avatar_gripper_description/meshes/${prefix}/thumb_knuckle.STL"/>
-        </geometry>
-        <material name="">
-          <color rgba="0.9 0.9 0.9 1"/>
-        </material>
-      </visual>
-      <collision>
-        <origin xyz="0 0 0" rpy="0 0 0"/>
-        <geometry>
-          <mesh filename="package://avatar_gripper_description/meshes/${prefix}/thumb_knuckle.STL"/>
-        </geometry>
-      </collision>
+          <mesh filename="package://avatar_gripper_description/meshes/${prefix}/thumb_knuckle.obj"/>
+        </geometry>
+        <material name="">
+          <color rgba="0.9 0.9 0.9 1"/>
+        </material>
+      </visual>
+      <!-- <collision>
+        <origin xyz="0 0 0" rpy="0 0 0"/>
+        <geometry>
+          <mesh filename="package://avatar_gripper_description/meshes/${prefix}/thumb_knuckle.obj"/>
+        </geometry>
+      </collision> -->
+      <xacro:collision_capsule_custom radius="0.009" length="0.047" xyz="0.0235 0 0" direction="x 0"/>
     </link>
   </xacro:macro>
@@ -79,16 +76,17 @@
         <origin xyz="0 0 0" rpy="0 0 0"/>
         <geometry>
-          <mesh filename="package://avatar_gripper_description/meshes/${prefix}/thumb_fingertip.STL"/>
-        </geometry>
-        <material name="">
-          <color rgba="0.9 0.9 0.9 1"/>
-        </material>
-      </visual>
-      <collision>
-        <origin xyz="0 0 0" rpy="0 0 0"/>
-        <geometry>
-          <mesh filename="package://avatar_gripper_description/meshes/${prefix}/thumb_fingertip.STL"/>
-        </geometry>
-      </collision>
+          <mesh filename="package://avatar_gripper_description/meshes/${prefix}/thumb_fingertip.obj"/>
+        </geometry>
+        <material name="">
+          <color rgba="0.9 0.9 0.9 1"/>
+        </material>
+      </visual>
+      <!-- <collision>
+        <origin xyz="0 0 0" rpy="0 0 0"/>
+        <geometry>
+          <mesh filename="package://avatar_gripper_description/meshes/${prefix}/thumb_fingertip.obj"/>
+        </geometry>
+      </collision> -->
+      <xacro:collision_capsule_custom radius="0.008" length="0.041" xyz="0.020 0 0" direction="x 0"/>
     </link>
   </xacro:macro>
@@ -102,5 +100,5 @@
         <origin xyz="0 0 0" rpy="0 0 0"/>
         <geometry>
-          <mesh filename="package://avatar_gripper_description/meshes/${prefix}/index_base_connector.STL"/>
+          <mesh filename="package://avatar_gripper_description/meshes/${prefix}/index_base_connector.obj"/>
         </geometry>
         <material name="">
@@ -111,5 +109,5 @@
         <origin xyz="0 0 0" rpy="0 0 0"/>
         <geometry>
-          <mesh filename="package://avatar_gripper_description/meshes/${prefix}/index_base_connector.STL"/>
+          <mesh filename="package://avatar_gripper_description/meshes/${prefix}/index_base_connector.obj"/>
         </geometry>
         <material name="">
@@ -128,16 +126,11 @@
         <origin xyz="0 0 0" rpy="0 0 0"/>
         <geometry>
-          <mesh filename="package://avatar_gripper_description/meshes/${prefix}/index_knuckle.STL"/>
-        </geometry>
-        <material name="">
-          <color rgba="0.9 0.9 0.9 1"/>
-        </material>
-      </visual>
-      <collision>
-        <origin xyz="0 0 0" rpy="0 0 0"/>
-        <geometry>
-          <mesh filename="package://avatar_gripper_description/meshes/${prefix}/index_knuckle.STL"/>
-        </geometry>
-      </collision>
+          <mesh filename="package://avatar_gripper_description/meshes/${prefix}/index_knuckle.obj"/>
+        </geometry>
+        <material name="">
+          <color rgba="0.9 0.9 0.9 1"/>
+        </material>
+      </visual>
+      <xacro:collision_capsule_custom radius="0.01" length="0.040" xyz="0.02 0 0" direction="x 0"/>
     </link>
   </xacro:macro>
@@ -151,16 +144,12 @@
         <origin xyz="0 0 0" rpy="0 0 0"/>
         <geometry>
-          <mesh filename="package://avatar_gripper_description/meshes/${prefix}/index_fingertip.STL"/>
-        </geometry>
-        <material name="">
-          <color rgba="0.9 0.9 0.9 1"/>
-        </material>
-      </visual>
-      <collision>
-        <origin xyz="0 0 0" rpy="0 0 0"/>
-        <geometry>
-          <mesh filename="package://avatar_gripper_description/meshes/${prefix}/index_fingertip.STL"/>
-        </geometry>
-      </collision>
+          <mesh filename="package://avatar_gripper_description/meshes/${prefix}/index_fingertip.obj"/>
+        </geometry>
+        <material name="">
+          <color rgba="0.9 0.9 0.9 1"/>
+        </material>
+      </visual>
+      <xacro:collision_capsule_custom radius="0.008" length="0.026" xyz="0.013 0 0" direction="x 0"/>
+      <xacro:collision_capsule_custom radius="0.008" length="0.023" xyz="0.038 -0.009 0" direction="x -0.67"/>
     </link>
   </xacro:macro>
@@ -174,16 +163,17 @@
         <origin xyz="0 0 0" rpy="0 0 0"/>
         <geometry>
-          <mesh filename="package://avatar_gripper_description/meshes/${prefix}/index_knuckle.STL"/>
-        </geometry>
-        <material name="">
-          <color rgba="0.9 0.9 0.9 1"/>
-        </material>
-      </visual>
-      <collision>
-        <origin xyz="0 0 0" rpy="0 0 0"/>
-        <geometry>
-          <mesh filename="package://avatar_gripper_description/meshes/${prefix}/index_knuckle.STL"/>
-        </geometry>
-      </collision>
+          <mesh filename="package://avatar_gripper_description/meshes/${prefix}/index_knuckle.obj"/>
+        </geometry>
+        <material name="">
+          <color rgba="0.9 0.9 0.9 1"/>
+        </material>
+      </visual>
+      <!-- <collision>
+        <origin xyz="0 0 0" rpy="0 0 0"/>
+        <geometry>
+          <mesh filename="package://avatar_gripper_description/meshes/${prefix}/index_knuckle.obj"/>
+        </geometry>
+      </collision> -->
+      <xacro:collision_capsule_custom radius="0.01" length="0.040" xyz="0.02 0 0" direction="x 0"/>
     </link>
   </xacro:macro>
@@ -197,16 +187,18 @@
         <origin xyz="0 0 0" rpy="0 0 0"/>
         <geometry>
-          <mesh filename="package://avatar_gripper_description/meshes/${prefix}/index_fingertip.STL"/>
-        </geometry>
-        <material name="">
-          <color rgba="0.9 0.9 0.9 1"/>
-        </material>
-      </visual>
-      <collision>
-        <origin xyz="0 0 0" rpy="0 0 0"/>
-        <geometry>
-          <mesh filename="package://avatar_gripper_description/meshes/${prefix}/index_fingertip.STL"/>
-        </geometry>
-      </collision>
+          <mesh filename="package://avatar_gripper_description/meshes/${prefix}/index_fingertip.obj"/>
+        </geometry>
+        <material name="">
+          <color rgba="0.9 0.9 0.9 1"/>
+        </material>
+      </visual>
+      <!-- <collision>
+        <origin xyz="0 0 0" rpy="0 0 0"/>
+        <geometry>
+          <mesh filename="package://avatar_gripper_description/meshes/${prefix}/index_fingertip.obj"/>
+        </geometry>
+      </collision> -->
+      <xacro:collision_capsule_custom radius="0.008" length="0.026" xyz="0.013 0 0" direction="x 0"/>
+      <xacro:collision_capsule_custom radius="0.008" length="0.023" xyz="0.038 -0.009 0" direction="x -0.67"/>
     </link>
   </xacro:macro>
@@ -220,5 +212,5 @@
         <origin xyz="0 0 0" rpy="0 0 0"/>
         <geometry>
-          <mesh filename="package://avatar_gripper_description/meshes/${prefix}/thumb_swivel_link.STL"/>
+          <mesh filename="package://avatar_gripper_description/meshes/${prefix}/thumb_swivel_link.obj"/>
         </geometry>
         <material name="">
@@ -229,5 +221,5 @@
         <origin xyz="0 0 0" rpy="0 0 0"/>
         <geometry>
-          <mesh filename="package://avatar_gripper_description/meshes/${prefix}/thumb_swivel_link.STL"/>
+          <mesh filename="package://avatar_gripper_description/meshes/${prefix}/thumb_swivel_link.obj"/>
         </geometry>
       </collision>
@@ -237,5 +229,5 @@
   <xacro:macro name="thumb_knuckle_joint" params="prefix">
     <joint name="${prefix}_thumb_knuckle_joint" type="revolute">
-      <origin xyz="0 0 0" rpy="0 2.75 0"/>
+      <origin xyz="0 0 0" rpy="0 3.064 0"/>
       <parent link="${prefix}_thumb_base"/>
       <child link="${prefix}_thumb_knuckle"/>
@@ -249,5 +241,6 @@
   <xacro:macro name="thumb_finger_joint" params="prefix">
     <joint name="${prefix}_thumb_finger_joint" type="revolute">
-      <origin xyz="0.04568 0 0.01106" rpy="0 0.57 0"/>
+      <!-- <origin xyz="0.04568 0 0.01106" rpy="0 0.57 0"/> -->
+      <origin xyz="0.047 0 0" rpy="0 ${0.57-40/180*pi} 0"/>
       <parent link="${prefix}_thumb_knuckle"/>
       <child link="${prefix}_thumb_finger"/>
@@ -261,5 +254,5 @@
   <xacro:macro name="thumb_base_swivel_joint" params="prefix">
     <joint name="${prefix}_thumb_base_swivel_joint" type="fixed">
-      <origin xyz="-0.03742 0 0.05089" rpy="0 0 0"/>
+      <origin xyz="-0.03742 0 0.05089" rpy="0 -${30/180*pi} 0"/>
       <parent link="${prefix}_thumb_swivel_link"/>
       <child link="${prefix}_thumb_base"/>
@@ -286,8 +279,8 @@
     <joint name="${prefix}_index_knuckle_joint" type="revolute">
       <xacro:if value="${prefix == 'left'}">
-        <origin xyz="+0.021564878 0.008545 -0.0024358" rpy="1.19730672 1.07478656 1.15162329"/>
+        <origin xyz="0.02156 0.008545 -0.0024358" rpy="-0.8363 1.3087 -0.9408"/>
       </xacro:if>
       <xacro:if value="${prefix == 'right'}">
-        <origin xyz="-0.021564878 0.008545 -0.0024358" rpy="1.94428593 1.07478656 1.98996937"/>
+        <origin xyz="-0.021564878 0.008545 -0.0024358" rpy="-2.3053 1.3087 -2.2008"/>
       </xacro:if>
       <parent link="${prefix}_index_base_connector"/>
@@ -302,5 +295,5 @@
   <xacro:macro name="index_fingertip_joint" params="prefix">
     <joint name="${prefix}_index_fingertip_joint" type="revolute">
-      <origin xyz="0.0353829 -0.02780 0" rpy="0 0 -0.35"/>
+      <origin xyz="0.04499 0 0" rpy="0 0 0.313"/>
       <parent link="${prefix}_index_knuckle"/>
       <child link="${prefix}_index_fingertip"/>
@@ -315,8 +308,8 @@
     <joint name="${prefix}_middle_knuckle_joint" type="revolute">
       <xacro:if value="${prefix == 'left'}">
-        <origin xyz="-0.02156 0.008545 -0.0024358" rpy="1.94428593 1.07478656 1.98996937"/>
+        <origin xyz="-0.021564878 0.008545 -0.0024358" rpy="-2.3053 1.3087 -2.2008"/>
       </xacro:if>
       <xacro:if value="${prefix == 'right'}">
-        <origin xyz="0.02156 0.008545 -0.0024358" rpy="1.19730672 1.07478656 1.15162329"/>
+        <origin xyz="0.02156 0.008545 -0.0024358" rpy="-0.8363 1.3087 -0.9408"/>
       </xacro:if>
       <parent link="${prefix}_index_base_connector"/>
@@ -331,5 +324,5 @@
   <xacro:macro name="middle_fingertip_joint" params="prefix">
     <joint name="${prefix}_middle_fingertip_joint" type="revolute">
-      <origin xyz="0.0353829 -0.02780 0" rpy="0 0 -0.35"/>
+      <origin xyz="0.04499 0 0" rpy="0 0 0.313"/>
       <parent link="${prefix}_middle_knuckle"/>
       <child link="${prefix}_middle_fingertip"/>

File: avatar_gripper_description/urdf/avatar_gripper_right.urdf (robot description, URDF)
Before this commit: robot avatar_gripper_3f_model, 13 links, 12 joints
Links:
- link right_gripper_base: geometry visual mesh filename=package://avatar_gripper_description/meshes/right/gripper_b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
- link right_index_fingertip: geometry collision cylinder length=0.023 radius=0.008; collision cylinder length=0.026 radius=0.008
- link right_index_knuckle: geometry collision cylinder length=0.04 radius=0.01; collision sphere radius=0.01
- link right_middle_fingertip: geometry collision cylinder length=0.023 radius=0.008; collision cylinder length=0.026 radius=0.008
- link right_middle_knuckle: geometry collision cylinder length=0.04 radius=0.01; collision sphere radius=0.01
- link right_thumb_base: geometry collision cylinder length=0.036 radius=0.01; collision sphere radius=0.01
- link right_thumb_finger: geometry collision cylinder length=0.041 radius=0.008; collision sphere radius=0.008
- link right_thumb_knuckle: geometry collision cylinder length=0.047 radius=0.009; collision sphere radius=0.009
Joints:
- joint right_index_fingertip_joint: origin xyz=0.0353829 -0.02780 0 rpy=0 0 -0.35 -> xyz=0.04499 0 0 rpy=0 0 0.313
- joint right_index_knuckle_joint: origin xyz=-0.021564878 0.008545 -0.0024358 rpy=1.94428593 1.07478656 1.98996937 -> xyz=-0.021564878 0.008545 -0.0024358 rpy=-2.3053 1.3087 -2.2008
- joint right_middle_fingertip_joint: origin xyz=0.0353829 -0.02780 0 rpy=0 0 -0.35 -> xyz=0.04499 0 0 rpy=0 0 0.313
- joint right_middle_knuckle_joint: origin xyz=0.02156 0.008545 -0.0024358 rpy=1.19730672 1.07478656 1.15162329 -> xyz=0.02156 0.008545 -0.0024358 rpy=-0.8363 1.3087 -0.9408
- joint right_thumb_base_swivel_joint: origin xyz=-0.03742 0 0.05089 rpy=0 0 0 -> xyz=-0.03742 0 0.05089 rpy=0 -0.5235987755982988 0
- joint right_thumb_finger_joint: origin xyz=0.04568 0 0.01106 rpy=0 0.57 0 -> xyz=0.047 0 0 rpy=0 -0.12813170079773184 0
- joint right_thumb_knuckle_joint: origin xyz=0 0 0 rpy=0 2.75 0 -> xyz=0 0 0 rpy=0 3.064 0

File: avatar_gripper_description/urdf/avatar_gripper_right_nomimic.urdf (robot description, URDF)
Before this commit: robot avatar_gripper_3f_model, 13 links, 12 joints
Links:
- link right_gripper_base: geometry visual mesh filename=package://avatar_gripper_description/meshes/right/gripper_b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
- link right_index_fingertip: geometry collision cylinder length=0.023 radius=0.008; collision cylinder length=0.026 radius=0.008
- link right_index_knuckle: geometry collision cylinder length=0.04 radius=0.01; collision sphere radius=0.01
- link right_middle_fingertip: geometry collision cylinder length=0.023 radius=0.008; collision cylinder length=0.026 radius=0.008
- link right_middle_knuckle: geometry collision cylinder length=0.04 radius=0.01; collision sphere radius=0.01
- link right_thumb_base: geometry collision cylinder length=0.036 radius=0.01; collision sphere radius=0.01
- link right_thumb_finger: geometry collision cylinder length=0.041 radius=0.008; collision sphere radius=0.008
- link right_thumb_knuckle: geometry collision cylinder length=0.047 radius=0.009; collision sphere radius=0.009
Joints:
- joint right_index_fingertip_joint: origin xyz=0.0353829 -0.02780 0 rpy=0 0 -0.35 -> xyz=0.04499 0 0 rpy=0 0 0.313
- joint right_index_knuckle_joint: origin xyz=-0.021564878 0.008545 -0.0024358 rpy=1.94428593 1.07478656 1.98996937 -> xyz=-0.021564878 0.008545 -0.0024358 rpy=-2.3053 1.3087 -2.2008
- joint right_middle_fingertip_joint: origin xyz=0.0353829 -0.02780 0 rpy=0 0 -0.35 -> xyz=0.04499 0 0 rpy=0 0 0.313
- joint right_middle_knuckle_joint: origin xyz=0.02156 0.008545 -0.0024358 rpy=1.19730672 1.07478656 1.15162329 -> xyz=0.02156 0.008545 -0.0024358 rpy=-0.8363 1.3087 -0.9408
- joint right_thumb_base_swivel_joint: origin xyz=-0.03742 0 0.05089 rpy=0 0 0 -> xyz=-0.03742 0 0.05089 rpy=0 -0.5235987755982988 0
- joint right_thumb_finger_joint: origin xyz=0.04568 0 0.01106 rpy=0 0.57 0 -> xyz=0.047 0 0 rpy=0 -0.12813170079773184 0
- joint right_thumb_knuckle_joint: origin xyz=0 0 0 rpy=0 2.75 0 -> xyz=0 0 0 rpy=0 3.064 0

File: avatar_robot_description/urdf/dual_panda_with_gripper.urdf (robot description, URDF)
Before this commit: robot avatar, 67 links, 66 joints
Links:
- link left_gripper_base: geometry visual mesh filename=package://avatar_gripper_description/meshes/left/gripper_ba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
- link left_index_fingertip: geometry collision cylinder length=0.023 radius=0.008; collision cylinder length=0.026 radius=0.008
- link left_index_knuckle: geometry collision cylinder length=0.04 radius=0.01; collision sphere radius=0.01
- link left_middle_fingertip: geometry collision cylinder length=0.023 radius=0.008; collision cylinder length=0.026 radius=0.008
- link left_middle_knuckle: geometry collision cylinder length=0.04 radius=0.01; collision sphere radius=0.01
- link left_thumb_base: geometry collision cylinder length=0.036 radius=0.01; collision sphere radius=0.01
- link left_thumb_finger: geometry collision cylinder length=0.041 radius=0.008; collision sphere radius=0.008
- link left_thumb_knuckle: geometry collision cylinder length=0.047 radius=0.009; collision sphere radius=0.009
- link right_gripper_base: geometry visual mesh filename=package://avatar_gripper_description/meshes/right/gripper_b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
- link right_index_fingertip: geometry collision cylinder length=0.023 radius=0.008; collision cylinder length=0.026 radius=0.008
- link right_index_knuckle: geometry collision cylinder length=0.04 radius=0.01; collision sphere radius=0.01
- link right_middle_fingertip: geometry collision cylinder length=0.023 radius=0.008; collision cylinder length=0.026 radius=0.008
- link right_middle_knuckle: geometry collision cylinder length=0.04 radius=0.01; collision sphere radius=0.01
- link right_thumb_base: geometry collision cylinder length=0.036 radius=0.01; collision sphere radius=0.01
- link right_thumb_finger: geometry collision cylinder length=0.041 radius=0.008; collision sphere radius=0.008
- link right_thumb_knuckle: geometry collision cylinder length=0.047 radius=0.009; collision sphere radius=0.009
Joints:
- joint left_index_fingertip_joint: origin xyz=0.0353829 -0.02780 0 rpy=0 0 -0.35 -> xyz=0.04499 0 0 rpy=0 0 0.313
- joint left_index_knuckle_joint: origin xyz=+0.021564878 0.008545 -0.0024358 rpy=1.19730672 1.07478656 1.15162329 -> xyz=0.02156 0.008545 -0.0024358 rpy=-0.8363 1.3087 -0.9408
- joint left_middle_fingertip_joint: origin xyz=0.0353829 -0.02780 0 rpy=0 0 -0.35 -> xyz=0.04499 0 0 rpy=0 0 0.313
- joint left_middle_knuckle_joint: origin xyz=-0.02156 0.008545 -0.0024358 rpy=1.94428593 1.07478656 1.98996937 -> xyz=-0.021564878 0.008545 -0.0024358 rpy=-2.3053 1.3087 -2.2008
- joint left_thumb_base_swivel_joint: origin xyz=-0.03742 0 0.05089 rpy=0 0 0 -> xyz=-0.03742 0 0.05089 rpy=0 -0.5235987755982988 0
- joint left_thumb_finger_joint: origin xyz=0.04568 0 0.01106 rpy=0 0.57 0 -> xyz=0.047 0 0 rpy=0 -0.12813170079773184 0
- joint left_thumb_knuckle_joint: origin xyz=0 0 0 rpy=0 2.75 0 -> xyz=0 0 0 rpy=0 3.064 0
- joint right_index_fingertip_joint: origin xyz=0.0353829 -0.02780 0 rpy=0 0 -0.35 -> xyz=0.04499 0 0 rpy=0 0 0.313
- joint right_index_knuckle_joint: origin xyz=-0.021564878 0.008545 -0.0024358 rpy=1.94428593 1.07478656 1.98996937 -> xyz=-0.021564878 0.008545 -0.0024358 rpy=-2.3053 1.3087 -2.2008
- joint right_middle_fingertip_joint: origin xyz=0.0353829 -0.02780 0 rpy=0 0 -0.35 -> xyz=0.04499 0 0 rpy=0 0 0.313
- joint right_middle_knuckle_joint: origin xyz=0.02156 0.008545 -0.0024358 rpy=1.19730672 1.07478656 1.15162329 -> xyz=0.02156 0.008545 -0.0024358 rpy=-0.8363 1.3087 -0.9408
- joint right_thumb_base_swivel_joint: origin xyz=-0.03742 0 0.05089 rpy=0 0 0 -> xyz=-0.03742 0 0.05089 rpy=0 -0.5235987755982988 0
- joint right_thumb_finger_joint: origin xyz=0.04568 0 0.01106 rpy=0 0.57 0 -> xyz=0.047 0 0 rpy=0 -0.12813170079773184 0
- joint right_thumb_knuckle_joint: origin xyz=0 0 0 rpy=0 2.75 0 -> xyz=0 0 0 rpy=0 3.064 0
