Commit message: replaced all mesh collision file for gripper with capsule collision primitive

File: avatar_robot_description/urdf/dual_panda_with_gripper_nomimic.urdf (robot description, URDF)
Before this commit: robot avatar, 67 links, 66 joints
Links:
- link left_gripper_base: geometry visual mesh filename=package://avatar_gripper_description/meshes/left/gripper_ba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
- link left_index_fingertip: geometry collision cylinder length=0.023 radius=0.008; collision cylinder length=0.026 radius=0.008
- link left_index_knuckle: geometry collision cylinder length=0.04 radius=0.01; collision sphere radius=0.01
- link left_middle_fingertip: geometry collision cylinder length=0.023 radius=0.008; collision cylinder length=0.026 radius=0.008
- link left_middle_knuckle: geometry collision cylinder length=0.04 radius=0.01; collision sphere radius=0.01
- link left_thumb_base: geometry collision cylinder length=0.036 radius=0.01; collision sphere radius=0.01
- link left_thumb_finger: geometry collision cylinder length=0.041 radius=0.008; collision sphere radius=0.008
- link left_thumb_knuckle: geometry collision cylinder length=0.047 radius=0.009; collision sphere radius=0.009
- link right_gripper_base: geometry visual mesh filename=package://avatar_gripper_description/meshes/right/gripper_b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
- link right_index_fingertip: geometry collision cylinder length=0.023 radius=0.008; collision cylinder length=0.026 radius=0.008
- link right_index_knuckle: geometry collision cylinder length=0.04 radius=0.01; collision sphere radius=0.01
- link right_middle_fingertip: geometry collision cylinder length=0.023 radius=0.008; collision cylinder length=0.026 radius=0.008
- link right_middle_knuckle: geometry collision cylinder length=0.04 radius=0.01; collision sphere radius=0.01
- link right_thumb_base: geometry collision cylinder length=0.036 radius=0.01; collision sphere radius=0.01
- link right_thumb_finger: geometry collision cylinder length=0.041 radius=0.008; collision sphere radius=0.008
- link right_thumb_knuckle: geometry collision cylinder length=0.047 radius=0.009; collision sphere radius=0.009
Joints:
- joint left_index_fingertip_joint: origin xyz=0.0353829 -0.02780 0 rpy=0 0 -0.35 -> xyz=0.04499 0 0 rpy=0 0 0.313
- joint left_index_knuckle_joint: origin xyz=+0.021564878 0.008545 -0.0024358 rpy=1.19730672 1.07478656 1.15162329 -> xyz=0.02156 0.008545 -0.0024358 rpy=-0.8363 1.3087 -0.9408
- joint left_middle_fingertip_joint: origin xyz=0.0353829 -0.02780 0 rpy=0 0 -0.35 -> xyz=0.04499 0 0 rpy=0 0 0.313
- joint left_middle_knuckle_joint: origin xyz=-0.02156 0.008545 -0.0024358 rpy=1.94428593 1.07478656 1.98996937 -> xyz=-0.021564878 0.008545 -0.0024358 rpy=-2.3053 1.3087 -2.2008
- joint left_thumb_base_swivel_joint: origin xyz=-0.03742 0 0.05089 rpy=0 0 0 -> xyz=-0.03742 0 0.05089 rpy=0 -0.5235987755982988 0
- joint left_thumb_finger_joint: origin xyz=0.04568 0 0.01106 rpy=0 0.57 0 -> xyz=0.047 0 0 rpy=0 -0.12813170079773184 0
- joint left_thumb_knuckle_joint: origin xyz=0 0 0 rpy=0 2.75 0 -> xyz=0 0 0 rpy=0 3.064 0
- joint right_index_fingertip_joint: origin xyz=0.0353829 -0.02780 0 rpy=0 0 -0.35 -> xyz=0.04499 0 0 rpy=0 0 0.313
- joint right_index_knuckle_joint: origin xyz=-0.021564878 0.008545 -0.0024358 rpy=1.94428593 1.07478656 1.98996937 -> xyz=-0.021564878 0.008545 -0.0024358 rpy=-2.3053 1.3087 -2.2008
- joint right_middle_fingertip_joint: origin xyz=0.0353829 -0.02780 0 rpy=0 0 -0.35 -> xyz=0.04499 0 0 rpy=0 0 0.313
- joint right_middle_knuckle_joint: origin xyz=0.02156 0.008545 -0.0024358 rpy=1.19730672 1.07478656 1.15162329 -> xyz=0.02156 0.008545 -0.0024358 rpy=-0.8363 1.3087 -0.9408
- joint right_thumb_base_swivel_joint: origin xyz=-0.03742 0 0.05089 rpy=0 0 0 -> xyz=-0.03742 0 0.05089 rpy=0 -0.5235987755982988 0
- joint right_thumb_finger_joint: origin xyz=0.04568 0 0.01106 rpy=0 0.57 0 -> xyz=0.047 0 0 rpy=0 -0.12813170079773184 0
- joint right_thumb_knuckle_joint: origin xyz=0 0 0 rpy=0 2.75 0 -> xyz=0 0 0 rpy=0 3.064 0

Commit message: added transmission definition of the gripper motor

File: avatar_gripper_description/urdf/avatar_gripper_3f_macro.xacro (robot description, xacro)
@@ -388,4 +388,16 @@
       <limit lower="-2.3" upper="-0.05" velocity="2.0" effort="1000" />
     </joint>
+  </xacro:macro>
+  <xacro:macro name="gripper_motor_transmission" params="prefix name">
+    <transmission name="${prefix}_${name}_transmission">
+      <type>transmission_interface/SimpleTransmission</type>
+      <joint name="${prefix}_${name}">
+        <hardwareInterface>PositionJointInterface</hardwareInterface>
+      </joint>
+      <actuator name="${prefix}_${name}_actuator">
+        <hardwareInterface>PositionJointInterface</hardwareInterface>
+        <mechanicalReduction>1</mechanicalReduction>
+      </actuator>
+    </transmission>
   </xacro:macro>
   <xacro:macro name="avatar_gripper_3f" params="prefix motor_base_attach_to">
@@ -415,4 +427,14 @@
     <xacro:motor_link prefix="${prefix}" actuation="index_flex"/>
     <xacro:index_flex_motor_joint prefix="${prefix}" motor_base_attach_to="${motor_base_attach_to}"/>
+    <xacro:gripper_motor_transmission prefix="${prefix}" name="thumb_knuckle_joint"/>
+    <xacro:gripper_motor_transmission prefix="${prefix}" name="thumb_finger_joint"/>
+    <xacro:gripper_motor_transmission prefix="${prefix}" name="thumb_swivel_joint"/>
+    <xacro:gripper_motor_transmission prefix="${prefix}" name="index_knuckle_joint"/>
+    <xacro:gripper_motor_transmission prefix="${prefix}" name="index_fingertip_joint"/>
+    <xacro:gripper_motor_transmission prefix="${prefix}" name="middle_knuckle_joint"/>
+    <xacro:gripper_motor_transmission prefix="${prefix}" name="middle_fingertip_joint"/>
+    <xacro:gripper_motor_transmission prefix="${prefix}" name="thumb_flex_motor_joint"/>
+    <xacro:gripper_motor_transmission prefix="${prefix}" name="thumb_swivel_motor_joint"/>
+    <xacro:gripper_motor_transmission prefix="${prefix}" name="index_flex_motor_joint"/>
   </xacro:macro>
 </robot>

Commit message: replaced collision model for index connector

File: avatar_gripper_description/urdf/avatar_gripper_3f_macro.xacro (robot description, xacro)
@@ -58,10 +58,4 @@
         </material>
       </visual>
-      <!-- <collision>
-        <origin xyz="0 0 0" rpy="0 0 0"/>
-        <geometry>
-          <mesh filename="package://avatar_gripper_description/meshes/${prefix}/thumb_knuckle.obj"/>
-        </geometry>
-      </collision> -->
       <xacro:collision_capsule_custom radius="0.009" length="0.047" xyz="0.0235 0 0" direction="x 0"/>
     </link>
@@ -82,10 +76,4 @@
         </material>
       </visual>
-      <!-- <collision>
-        <origin xyz="0 0 0" rpy="0 0 0"/>
-        <geometry>
-          <mesh filename="package://avatar_gripper_description/meshes/${prefix}/thumb_fingertip.obj"/>
-        </geometry>
-      </collision> -->
       <xacro:collision_capsule_custom radius="0.008" length="0.041" xyz="0.020 0 0" direction="x 0"/>
     </link>
@@ -107,11 +95,14 @@
       </visual>
       <collision>
-        <origin xyz="0 0 0" rpy="0 0 0"/>
-        <geometry>
-          <mesh filename="package://avatar_gripper_description/meshes/${prefix}/index_base_connector.obj"/>
-        </geometry>
-        <material name="">
-          <color rgba="0.9 0.9 0.9 1"/>
-        </material>
+        <origin xyz="-0.008 0 0.013" rpy="0 0 0"/>
+        <geometry>
+          <sphere radius="0.015"/>
+        </geometry>
+      </collision>
+      <collision>
+        <origin xyz="0.008 0 0.013" rpy="0 0 0"/>
+        <geometry>
+          <sphere radius="0.015"/>
+        </geometry>
       </collision>
     </link>
@@ -169,10 +160,4 @@
         </material>
       </visual>
-      <!-- <collision>
-        <origin xyz="0 0 0" rpy="0 0 0"/>
-        <geometry>
-          <mesh filename="package://avatar_gripper_description/meshes/${prefix}/index_knuckle.obj"/>
-        </geometry>
-      </collision> -->
       <xacro:collision_capsule_custom radius="0.01" length="0.040" xyz="0.02 0 0" direction="x 0"/>
     </link>
@@ -193,10 +178,4 @@
         </material>
       </visual>
-      <!-- <collision>
-        <origin xyz="0 0 0" rpy="0 0 0"/>
-        <geometry>
-          <mesh filename="package://avatar_gripper_description/meshes/${prefix}/index_fingertip.obj"/>
-        </geometry>
-      </collision> -->
       <xacro:collision_capsule_custom radius="0.008" length="0.026" xyz="0.013 0 0" direction="x 0"/>
       <xacro:collision_capsule_custom radius="0.008" length="0.023" xyz="0.038 -0.009 0" direction="x -0.67"/>
@@ -218,10 +197,4 @@
         </material>
       </visual>
-      <collision>
-        <origin xyz="0 0 0" rpy="0 0 0"/>
-        <geometry>
-          <mesh filename="package://avatar_gripper_description/meshes/${prefix}/thumb_swivel_link.obj"/>
-        </geometry>
-      </collision>
     </link>
   </xacro:macro>

File: avatar_gripper_description/urdf/avatar_gripper_right.urdf (robot description, URDF)
Before this commit: robot avatar_gripper_3f_model, 13 links, 12 joints
Links:
- link right_index_base_connector: geometry collision sphere radius=0.015; collision sphere radius=0.015
- link right_thumb_swivel_link: geometry visual mesh filename=package://avatar_gripper_description/meshes/right/thumb_swi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

File: avatar_gripper_description/urdf/avatar_gripper_right_nomimic.urdf (robot description, URDF)
Before this commit: robot avatar_gripper_3f_model, 13 links, 12 joints
Links:
- link right_index_base_connector: geometry collision sphere radius=0.015; collision sphere radius=0.015
- link right_thumb_swivel_link: geometry visual mesh filename=package://avatar_gripper_description/meshes/right/thumb_swi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
