Commit message: fixed typo

File: avatar_robot_description/franka/panda/panda_with_gripper.urdf (robot description, URDF)
Before this commit: robot panda, 30 links, 29 joints
Joints:
- joint right_index_fingertip_joint: mimic joint=right_index_flex_motor_joint multiplier=0.4 -> joint=right_index_flex_motor_joint multiplier=0.4 offset=0
- joint right_index_knuckle_joint: mimic joint=right_index_flex_motor_joint multiplier=0.4016 -> joint=right_index_flex_motor_joint multiplier=0.4016 offset=0
- joint right_thumb_finger_joint: mimic joint=right_thumb_flex_motor_joint multiplier=0.24 -> joint=right_thumb_flex_motor_joint multiplier=0.24 offset=0
- joint right_thumb_knuckle_joint: mimic joint=right_thumb_flex_motor_joint multiplier=0.28 -> joint=right_thumb_flex_motor_joint multiplier=0.28 offset=0
